File: engine-board/engine-board.kicad_pcb (KiCad board)
At the start: 2 copper layers, 304.1 x 76.2 mm, 61 parts, among them J1 MAXON Pump Controller, J10 USB/SER/CHRGR, J11 Pump Current Sensor, J12 Steering Turbines, J2 Power Rail, J24 Battery Input, J27 Leak Sensor, J31 Solenoid, J32 Solenoid Current Sensor, J33 BME280 Sensor, J34 RV1805 Clock, J35 Reservoir Pressure Sensor, J36 Bladder Pressure Sensor, J37 VL6180 Range Sensor, J42 HMC6343 COMPASS, J43 NEO08MU GPS, J44 Turbine Current Sensor, J45 Engine Current Sensor, J47 QWIIC 1, J48 QWIIC 2, J50 SD Card, J53 Switch Bulkhead, J61 Turbine 1 ESC, J62 Turbine 2 ESC, Q1 IRLB8721PBF, U1 FEATHER_M0_BASIC_PROTO, U10 Pololu_2812, U2 R-78B5.0-2.0, U3 R-78B3.3-2.0, U4 Teensy4.1, U51 IMU_BN0080

Commit message: Broke up into multiple schematics
- broke up into multiple schematics
- replaced some parts based on availability of parts
Parts:
- removed J34: RV1805 Clock, Connector_Molex:Molex_KK-254_AE-6410-07A_1x07_P2.54mm_Vertical
- removed U4: Teensy4.1, Module:Teensy41
- added D301: 1N4001, Diode_THT:D_DO-41_SOD81_P10.16mm_Horizontal, F.Cu at (100.8, 229.9)
- added J101: SD Card, Connector_Molex:Molex_KK-254_AE-6410-08A_1x08_P2.54mm_Vertical, F.Cu at (183.6, 259.9)
- added J201: Reservoir Pressure Sensor, TerminalBlock_CUI:CUI_TBP01R1W-508-04BE, F.Cu at (198.7, 195.1)
- added J202: Bladder Pressure Sensor, TerminalBlock_CUI:CUI_TBP01R1W-508-04BE, F.Cu at (198.7, 209.6)
- added J203: HMC6343 COMPASS, Connector_PinSocket_2.54mm:PinSocket_1x04_P2.54mm_Vertical, F.Cu at (240.7, 201.1)
- added J204: QWIIC 1, Connector_JST:JST_SH_BM04B-SRSS-TB_1x04-1MP_P1.00mm_Vertical, F.Cu at (194.8, 216.4)
- added J205: QWIIC 2, Connector_JST:JST_SH_BM04B-SRSS-TB_1x04-1MP_P1.00mm_Vertical, F.Cu at (203.6, 216.4)
- added J206: Leak Sensor, TerminalBlock_CUI:CUI_TBP01R1W-508-04BE, F.Cu at (230.8, 195.1)
- added J207: BME260 Sensor, Connector_PinSocket_2.54mm:PinSocket_1x04_P2.54mm_Vertical, F.Cu at (245.3, 201.1)
- added J208: RV1805 Clock, Connector_PinSocket_2.54mm:PinSocket_1x07_P2.54mm_Vertical, F.Cu at (228.6, 110.2)
- added J301: Steering Turbines, Connector_Molex:Molex_Micro-Fit_3.0_43045-0821_2x04-1MP_P3.00mm_Horizontal, F.Cu at (156.2, 223.2)
- added J302: MAXON Pump Controller, TerminalBlock_CUI:CUI_TBP01R1W-508-12BE, F.Cu at (107.4, 195.1)
- added J303: Pump Current Sensor, Connector_PinSocket_2.54mm:PinSocket_1x06_P2.54mm_Vertical, F.Cu at (175.5, 204.0)
- added J304: VL6180 Range Sensor, Connector_PinSocket_2.54mm:PinSocket_1x06_P2.54mm_Vertical, F.Cu at (184.7, 186.7)
- added J305: Turbine 1 ESC, TerminalBlock_CUI:CUI_TBP01R1W-508-08BE, F.Cu at (107.4, 224.1)
- added J306: Turbine 2 ESC, TerminalBlock_CUI:CUI_TBP01R1W-508-08BE, F.Cu at (107.4, 209.6)
- added J307: Turbine Current Sensor, Connector_PinSocket_2.54mm:PinSocket_1x06_P2.54mm_Vertical, F.Cu at (180.1, 186.7)
- added J308: Solenoid Current Sensor, Connector_PinSocket_2.54mm:PinSocket_1x06_P2.54mm_Vertical, F.Cu at (175.5, 186.7)
- added J309: Solenoid, TerminalBlock_CUI:CUI_TBP01R1W-508-02BE, F.Cu at (159.7, 209.6)
- added J401: USB/SER/CHRGR, Connector_Molex:Molex_Micro-Fit_3.0_43045-1600_2x08_P3.00mm_Horizontal, F.Cu at (103.6, 261.5)
- added J402: Power Rail, Connector_PinSocket_2.54mm:PinSocket_1x08_P2.54mm_Vertical, F.Cu at (174.0, 239.4)
- added J403: INA219 Engine Current Sensor, Connector_PinSocket_2.54mm:PinSocket_1x06_P2.54mm_Vertical, F.Cu at (162.6, 253.8)
- added J404: Switch Bulkhead, TerminalBlock_CUI:CUI_TBP01R1W-508-02BE, F.Cu at (137.6, 262.3)
- added J405: Battery Input, TerminalBlock_CUI:CUI_TBP01R1W-508-12BE, F.Cu at (107.4, 247.8)
- added J406: 3V Current Sensor, Connector_PinSocket_2.54mm:PinSocket_1x06_P2.54mm_Vertical, F.Cu at (158.0, 253.8)
- added J407: 5V Current Sensor, Connector_PinSocket_2.54mm:PinSocket_1x06_P2.54mm_Vertical, F.Cu at (153.4, 261.8)
- added J46: 3V Current Sensor, Connector_Molex:Molex_KK-254_AE-6410-06A_1x06_P2.54mm_Vertical, F.Cu at (122.9, 132.6)
- added J501: Serial Telemetry, TerminalBlock_CUI:CUI_TBP01R1W-508-04BE, F.Cu at (258.9, 236.7)
- added J502: NEO08MU GPS, Connector_PinSocket_2.54mm:PinSocket_1x08_P2.54mm_Vertical, F.Cu at (284.9, 228.3)
- added J503: RockBLOCK 9603, Connector_PinSocket_2.54mm:PinSocket_1x06_P2.54mm_Vertical, F.Cu at (289.5, 228.3)
- added J62: Engine Current Sensor, Connector_Molex:Molex_KK-254_AE-6410-06A_1x06_P2.54mm_Vertical, F.Cu at (86.4, 137.9)
- added J64: Serial Telemetry, TerminalBlock_CUI:CUI_TBP01R1W-508-04BE, F.Cu at (89.9, 99.1)
- added JP101: PumpAngGND, Jumper:SolderJumper-2_P1.3mm_Open_Pad1.0x1.5mm, F.Cu at (205.9, 257.8)
- added JP202: IMU ADR Jump, Connector_PinHeader_2.54mm:PinHeader_1x02_P2.54mm_Vertical, F.Cu at (210.4, 215.6)
- added Q301: IRLB8721PBF, Package_TO_SOT_THT:TO-220-3_Vertical, F.Cu at (116.1, 231.7)
- added R201: 1kohm, Resistor_THT:R_Axial_DIN0204_L3.6mm_D1.6mm_P5.08mm_Vertical, F.Cu at (191.9, 221.1)
- added R202: 2kohm, Resistor_THT:R_Axial_DIN0204_L3.6mm_D1.6mm_P5.08mm_Vertical, F.Cu at (200.1, 221.1)
- added R301: 10kohm, Resistor_THT:R_Axial_DIN0204_L3.6mm_D1.6mm_P5.08mm_Vertical, F.Cu at (126.0, 229.3)
- added TP201: raw leak, TestPoint:TestPoint_THTPad_3.0x3.0mm_Drill1.5mm, F.Cu at (215.2, 215.8)
- added TP202: leak3v3, TestPoint:TestPoint_THTPad_3.0x3.0mm_Drill1.5mm, F.Cu at (250.1, 201.3)
- added U101: Teensy3.6_All_Pins, Symbol:Teensy35_36, F.Cu at (328.4, 121.2)
- added U202: BN0055, Sensor_Motion:ADA_BN0055, F.Cu at (230.4, 209.8)
- added U402: R-78B3.3-2.0, Converter_DCDC:Converter_DCDC_RECOM_R-78B-2.0_THT, F.Cu at (103.0, 269.1)
- added U403: R-78B5.0-2.0, Converter_DCDC:Converter_DCDC_RECOM_R-78B-2.0_THT, F.Cu at (116.2, 269.1)
- J45: value Engine Current Sensor -> 5V Current Sensor
- J47, J48: footprint Connector_Molex:Molex_KK-254_AE-6410-04A_1x04_P2.54mm_Vertical -> Connector_JST:JST_SH_BM04B-SRSS-TB_1x04-1MP_P1.00mm_Vertical
- moved U3 68.9 mm to (185.9, 103.9)
- moved U2 61.3 mm to (185.7, 92.2)
- moved J45 40.0 mm to (123.2, 122.9)
- moved Q1 19.7 mm to (169.7, 94.2)
- moved J48 10.2 mm to (90.2, 159.8)
- moved J47 7.12 mm to (80.5, 159.8)
- renumbered J62 to J60, JP1 to JP102, JP50 to JP103, JP51 to JP104, R2 to R101, R1 to R102, U1 to U102
Connections:
- J11 pad 1: /i2c_scl_1 -> +3V3
- J11 pad 2: /i2c_sda_1 -> -BATT
- J11 pad 3: +3V3 -> /i2c_scl_1
- J11 pad 4: -BATT -> /i2c_sda_1
- J11 pad 6: -BATT -> +BATT
- J2 pad 6: Net-(J2-Pad6) -> /switched_BATT+
- J24 pad 1: Net-(J24-Pad1) -> /raw_BATT+
- J24 pad 2: Net-(J24-Pad1) -> /raw_BATT+
- J24 pad 3: Net-(J24-Pad3) -> /raw_BATT-
- J24 pad 4: Net-(J24-Pad3) -> /raw_BATT-
- J32 pad 1: /i2c_scl_1 -> +3V3
- J32 pad 2: /i2c_sda_1 -> -BATT
- J32 pad 3: +3V3 -> /i2c_scl_1
- J32 pad 4: -BATT -> /i2c_sda_1
- J32 pad 6: -BATT -> +BATT
- J44 pad 1: /i2c_scl_1 -> +3V3
- J44 pad 2: /i2c_sda_1 -> -BATT
- J44 pad 3: +3V3 -> /i2c_scl_1
- J44 pad 4: -BATT -> /i2c_sda_1
- J45 pad 1: /i2c_scl_1 -> +3V3
- J45 pad 2: /i2c_sda_1 -> -BATT
- J45 pad 3: +3V3 -> /i2c_scl_1
- J45 pad 4: -BATT -> /i2c_sda_1
- J45 pad 5: /engine_measured_BATT+ -> /5v_measured_BATT+
- J45 pad 6: -BATT -> +BATT
- U10 pad 1: +BATT -> /switched_BATT+
- U10 pad 2: +BATT -> /switched_BATT+
- U2 pad 1: +BATT -> /5v_measured_BATT+
- U3 pad 1: +BATT -> /3v_measured_BATT+
Other:
- net class power: clearance 0.2 -> 0.25; trace_width 1 -> 0.75; via_drill 0.4 -> 0.3

Commit message: pcb parts done, footprints updated, ready for routing
pre-routing step..
- finalized footprints
- verified layout, size, mounting holes (1.75" apart)
Parts:
- removed D2: 1N4001, Diode_THT:D_DO-41_SOD81_P10.16mm_Horizontal
- removed J11: Pump Current Sensor, Connector_Molex:Molex_KK-254_AE-6410-06A_1x06_P2.54mm_Vertical
- removed J2: Power Rail, Connector_Molex:Molex_KK-254_AE-6410-08A_1x08_P2.54mm_Vertical
- removed the J202 at (198.7, 209.6)
- removed the J206 at (230.8, 195.1)
- removed the J301 at (156.2, 223.2)
- removed J302: MAXON Pump Controller, TerminalBlock_CUI:CUI_TBP01R1W-508-12BE
- removed the J305 at (107.4, 224.1)
- removed the J306 at (107.4, 209.6)
- removed the J309 at (159.7, 209.6)
- removed J32: Solenoid Current Sensor, Connector_Molex:Molex_KK-254_AE-6410-06A_1x06_P2.54mm_Vertical
- removed J33: BME280 Sensor, Connector_Molex:Molex_KK-254_AE-6410-06A_1x06_P2.54mm_Vertical
- removed J35: Reservoir Pressure Sensor, TerminalBlock_CUI:CUI_TBP01R1W-508-04BE
- removed J37: VL6180 Range Sensor, Connector_Molex:Molex_KK-254_AE-6410-06A_1x06_P2.54mm_Vertical
- removed the J401 at (103.6, 261.5)
- removed the J404 at (137.6, 262.3)
- removed the J405 at (107.4, 247.8)
- removed J42: HMC6343 COMPASS, Connector_Molex:Molex_KK-254_AE-6410-04A_1x04_P2.54mm_Vertical
- removed J43: NEO08MU GPS, Connector_Molex:Molex_KK-254_AE-6410-08A_1x08_P2.54mm_Vertical
- removed J44: Turbine Current Sensor, Connector_Molex:Molex_KK-254_AE-6410-06A_1x06_P2.54mm_Vertical
- removed J45: 5V Current Sensor, Connector_Molex:Molex_KK-254_AE-6410-06A_1x06_P2.54mm_Vertical
- removed J46: 3V Current Sensor, Connector_Molex:Molex_KK-254_AE-6410-06A_1x06_P2.54mm_Vertical
- removed J47: QWIIC 1, Connector_JST:JST_SH_BM04B-SRSS-TB_1x04-1MP_P1.00mm_Vertical
- removed J48: QWIIC 2, Connector_JST:JST_SH_BM04B-SRSS-TB_1x04-1MP_P1.00mm_Vertical
- removed J50: SD Card, Connector_Molex:Molex_KK-254_AE-6410-08A_1x08_P2.54mm_Vertical
- removed the J501 at (258.9, 236.7)
- removed J62: Engine Current Sensor, Connector_Molex:Molex_KK-254_AE-6410-06A_1x06_P2.54mm_Vertical
- removed JP10: teensy_cw, Jumper:SolderJumper-2_P1.3mm_Open_Pad1.0x1.5mm
- removed JP11: pump_speed, Jumper:SolderJumper-2_P1.3mm_Open_Pad1.0x1.5mm
- removed JP12: pump_current, Jumper:SolderJumper-2_P1.3mm_Open_Pad1.0x1.5mm
- removed JP13: solenoid_gate, Jumper:SolderJumper-2_P1.3mm_Open_Pad1.0x1.5mm
- removed JP14: leak_in, Jumper:SolderJumper-2_P1.3mm_Open_Pad1.0x1.5mm
- removed JP15: imu_cs, Jumper:SolderJumper-2_P1.3mm_Open_Pad1.0x1.5mm
- removed JP202: IMU ADR Jump, Connector_PinHeader_2.54mm:PinHeader_1x02_P2.54mm_Vertical
- removed JP5: IMU PS1 Jump, Connector_PinHeader_2.54mm:PinHeader_1x02_P2.54mm_Vertical
- removed JP6: IMU PS0 Jump, Connector_PinHeader_2.54mm:PinHeader_1x02_P2.54mm_Vertical
- removed JP7: teensy_scl, Jumper:SolderJumper-2_P1.3mm_Open_Pad1.0x1.5mm
- removed JP8: teensy sda, Jumper:SolderJumper-2_P1.3mm_Open_Pad1.0x1.5mm
- removed JP9: teensy_ccw, Jumper:SolderJumper-2_P1.3mm_Open_Pad1.0x1.5mm
- removed Q1: IRLB8721PBF, Package_TO_SOT_THT:TO-220-3_Vertical
- removed R3: 10kohm, Resistor_THT:R_Axial_DIN0204_L3.6mm_D1.6mm_P5.08mm_Vertical
- removed R4: 1kohm, Resistor_THT:R_Axial_DIN0204_L3.6mm_D1.6mm_P5.08mm_Vertical
- removed R5: 2kohm, Resistor_THT:R_Axial_DIN0204_L3.6mm_D1.6mm_P5.08mm_Vertical
- removed TP1: raw leak, TestPoint:TestPoint_THTPad_3.0x3.0mm_Drill1.5mm
- removed TP2: leak3v3, TestPoint:TestPoint_THTPad_3.0x3.0mm_Drill1.5mm
- removed U10: Pololu_2812, Module:Pololu_SlidePwrSwitch
- removed the U402 at (103.0, 269.1)
- removed the U403 at (116.2, 269.1)
- removed U51: IMU_BN0080, Module:DIP-24_900_ELL
- added BT101: Battery_Cell, Battery:BatteryHolder_Keystone_1060_1x2032, F.Cu at (248.7, 128.3)
- added J504: RockBlock9603, Connector_PinSocket_2.54mm:PinSocket_1x10_P2.54mm_Vertical, F.Cu at (289.1, 139.7)
- added JP105: PumpAngGND, Jumper:SolderJumper-2_P1.3mm_Open_Pad1.0x1.5mm, F.Cu at (290.3, 124.7)
- added JP201: PumpAngGND, Jumper:SolderJumper-2_P1.3mm_Open_Pad1.0x1.5mm, F.Cu at (290.3, 131.2)
- added SW401: POWER, Module:SliderSwitch_Simple, F.Cu at (74.9, 161.8)
- added TP101: i2c_sda_1, TestPoint:TestPoint_Loop_D2.60mm_Drill1.6mm_Beaded, F.Cu at (266.6, 69.7)
- added TP102: i2c_scl_1, TestPoint:TestPoint_Loop_D2.60mm_Drill1.6mm_Beaded, F.Cu at (271.7, 69.7)
- added TP301: TP_SolGate, TestPoint:TestPoint_Loop_D2.60mm_Drill1.6mm_Beaded, F.Cu at (321.5, 37.5)
- added TP302: TP_SolVolt, TestPoint:TestPoint_Loop_D2.60mm_Drill1.6mm_Beaded, F.Cu at (326.5, 37.5)
- added TP304: TP_SolBat+, TestPoint:TestPoint_Loop_D2.60mm_Drill1.6mm_Beaded, F.Cu at (331.6, 37.5)
- added U401: Pololu_2814, Module:Pololu_Breakout-16_15.2x20.3mm, F.Cu at (82.0, 144.3)
- H1: renamed from REF1; value MountingHole_5.3mm_M5 -> MountingHole; footprint MountingHole:MountingHole_5.3mm_M5 -> MountingHole:MountingHole_5.3mm_M5_Pad
- H2: renamed from REF2; value MountingHole_5.3mm_M5 -> MountingHole; footprint MountingHole:MountingHole_5.3mm_M5 -> MountingHole:MountingHole_5.3mm_M5_Pad
- H3: renamed from REF3; value MountingHole_5.3mm_M5 -> MountingHole; footprint MountingHole:MountingHole_5.3mm_M5 -> MountingHole:MountingHole_5.3mm_M5_Pad
- H4: renamed from REF4; value MountingHole_5.3mm_M5 -> MountingHole; footprint MountingHole:MountingHole_5.3mm_M5 -> MountingHole:MountingHole_5.3mm_M5_Pad
- H5: renamed from REF5; value MountingHole_5.3mm_M5 -> MountingHole; footprint MountingHole:MountingHole_5.3mm_M5 -> MountingHole:MountingHole_5.3mm_M5_Pad
- H6: renamed from REF6; value MountingHole_5.3mm_M5 -> MountingHole; footprint MountingHole:MountingHole_5.3mm_M5 -> MountingHole:MountingHole_5.3mm_M5_Pad
- H7: renamed from REF7; value MountingHole_5.3mm_M5 -> MountingHole; footprint MountingHole:MountingHole_5.3mm_M5 -> MountingHole:MountingHole_5.3mm_M5_Pad
- H8: renamed from REF8; value MountingHole_5.3mm_M5 -> MountingHole; footprint MountingHole:MountingHole_5.3mm_M5 -> MountingHole:MountingHole_5.3mm_M5_Pad
- J101: footprint Connector_Molex:Molex_KK-254_AE-6410-08A_1x08_P2.54mm_Vertical -> Connector_PinSocket_2.54mm:PinSocket_1x08_P2.54mm_Vertical
- J303, J307, J308, J406, J407: footprint Connector_PinSocket_2.54mm:PinSocket_1x06_P2.54mm_Vertical -> Connector_PinSocket_2.54mm:PinSocket_1x08_P2.54mm_Vertical
- J403: value INA219 Engine Current Sensor -> Engine Current Sensor; footprint Connector_PinSocket_2.54mm:PinSocket_1x06_P2.54mm_Vertical -> Connector_PinSocket_2.54mm:PinSocket_1x08_P2.54mm_Vertical
- J503: footprint Connector_PinSocket_2.54mm:PinSocket_1x06_P2.54mm_Vertical -> Connector_PinSocket_2.54mm:PinSocket_1x10_P2.54mm_Vertical
- TP201: value raw leak -> TP_RawLeak; footprint TestPoint:TestPoint_THTPad_3.0x3.0mm_Drill1.5mm -> TestPoint:TestPoint_Loop_D2.60mm_Drill1.6mm_Beaded
- TP202: value leak3v3 -> TP_LeakSense; footprint TestPoint:TestPoint_THTPad_3.0x3.0mm_Drill1.5mm -> TestPoint:TestPoint_Loop_D2.60mm_Drill1.6mm_Beaded
- U202: value BN0055 -> BN0055 IMU
- moved J503 192.3 mm to (266.4, 37.3)
- moved J502 174.9 mm to (139.7, 130.8), turned to 90 degrees
- moved J204 172.2 mm to (74.1, 93.5)
- moved J205 172.2 mm to (83.0, 93.5)
- moved J101 164.5 mm to (296.2, 140.0)
- moved JP101 162.8 mm to (290.8, 118.9)
- moved J407 155.0 mm to (115.6, 111.5)
- moved J403 152.6 mm to (107.7, 111.5)
- moved J406 146.5 mm to (123.4, 111.5)
- moved J207 133.1 mm to (144.0, 114.8), turned to 90 degrees
- moved J303 129.0 mm to (85.6, 111.5)
- moved TP202 118.8 mm to (168.4, 115.1)
- moved Q301 118.5 mm to (168.2, 125.2)
- moved R301 118.5 mm to (178.1, 122.9)
- moved J308 111.6 mm to (93.0, 111.5)
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- renumbered J36 to J202, J27 to J206, J12 to J301, J61 to J305, J60 to J306, J31 to J309, J10 to J401, J53 to J404, J24 to J405, J64 to J501, U3 to U402, U2 to U403
Connections:
- net /Telemetry/irid_sleep renamed Net-(J503-Pad5)
- net Net-(U101-Pad56) renamed /irid_RI
- J1 pad 1: /pump_measured_BATT+ -> /Pump/pump_measured_BATT+
- J1 pad 2: /pump_measured_BATT+ -> /Pump/pump_measured_BATT+
- J206 pad 4: Net-(J27-Pad4) -> Net-(J206-Pad4)
- J301 pad 1: /turbine1_wht -> /Pump/turbine1_wht
- J301 pad 2: /turbine1_grn -> /Pump/turbine1_grn
- J301 pad 3: /turbine1_blu -> /Pump/turbine1_blu
- J301 pad 4: /external_switch_B -> /Pump/external_switch_B
- J301 pad 5: /turbine2_wht -> /Pump/turbine2_wht
- J301 pad 6: /turbine2_grn -> /Pump/turbine2_grn
- J301 pad 7: /turbine2_blu -> /Pump/turbine2_blu
- J301 pad 8: /external_switch_A -> /Pump/external_switch_A
- J303 pad 3: /Pump/i2c_scl_1 -> /i2c_scl_1
- J303 pad 4: /Pump/i2c_sda_1 -> /i2c_sda_1
- J303 pad 5: /Pump/pump_measured_BATT+ -> Net-(J303-Pad5)
- J304 pad 3: /Pump/i2c_scl_1 -> /i2c_scl_1
- J304 pad 4: /Pump/i2c_sda_1 -> /i2c_sda_1
- J305 pad 1: /turbine1_measured_pwr -> /Pump/turbine1_measured_pwr
- J305 pad 6: /turbine1_wht -> /Pump/turbine1_wht
- J305 pad 7: /turbine1_grn -> /Pump/turbine1_grn
- J305 pad 8: /turbine1_blu -> /Pump/turbine1_blu
- J306 pad 1: /turbine1_measured_pwr -> /Pump/turbine1_measured_pwr
- J306 pad 6: /turbine2_wht -> /Pump/turbine2_wht
- J306 pad 7: /turbine2_grn -> /Pump/turbine2_grn
- J306 pad 8: /turbine2_blu -> /Pump/turbine2_blu
- J307 pad 3: /Pump/i2c_scl_1 -> /i2c_scl_1
- J307 pad 4: /Pump/i2c_sda_1 -> /i2c_sda_1
- J307 pad 5: /Pump/turbine1_measured_pwr -> Net-(J307-Pad5)
- J308 pad 3: /Pump/i2c_scl_1 -> /i2c_scl_1
- J308 pad 4: /Pump/i2c_sda_1 -> /i2c_sda_1
- J308 pad 5: /Pump/solenoid_measured_BATT+ -> Net-(J308-Pad5)
- J309 pad 1: Net-(D2-Pad2) -> Net-(D301-Pad2)
- J309 pad 2: /solenoid_measured_BATT+ -> /Pump/solenoid_measured_BATT+
- J401 pad 10: /lipo_bat1_sense5 -> /Power/lipo_bat1_sense5
- J401 pad 11: /lipo_bat1_sense4 -> /Power/lipo_bat1_sense4
- J401 pad 12: /lipo_bat1_sense3 -> /Power/lipo_bat1_sense3
- J401 pad 13: /lipo_bat1_sense2 -> /Power/lipo_bat1_sense2
- J401 pad 14: /lipo_bat1_sense1 -> /Power/lipo_bat1_sense1
- J401 pad 15: /lipo_bat1_therm1 -> /Power/lipo_bat1_therm1
- J401 pad 16: /lipo_bat1_therm2 -> /Power/lipo_bat1_therm2
- J401 pad 4: /usb_pwr -> /Power/usb_pwr
- J401 pad 5: /usb_data_D0 -> /Power/usb_data_D0
- J401 pad 6: /usb_data_D1 -> /Power/usb_data_D1
- J401 pad 7: /rs232_tx -> /Power/rs232_tx
- J401 pad 8: /rs232_rx -> /Power/rs232_rx
- J401 pad 9: /rs232_gnd -> /Power/rs232_gnd
- J403 pad 5: /Power/switched_BATT+ -> Net-(J403-Pad5)
- J403 pad 6: +BATT -> /Power/switched_BATT+
- J404 pad 1: /external_switch_A -> /Power/external_switch_A
- J404 pad 2: /external_switch_B -> /Power/external_switch_B
- J405 pad 1: /raw_BATT+ -> /Power/raw_BATT+
- J405 pad 11: /lipo_bat_therm1 -> /Power/lipo_bat_therm1
- J405 pad 12: /lipo_bat_therm2 -> /Power/lipo_bat_therm2
- J405 pad 2: /raw_BATT+ -> /Power/raw_BATT+
- J405 pad 3: /raw_BATT- -> /Power/raw_BATT-
- J405 pad 4: /raw_BATT- -> /Power/raw_BATT-
- J405 pad 5: /lipo_bat1_sense1 -> /Power/lipo_bat1_sense1
- J405 pad 6: /lipo_bat1_sense2 -> /Power/lipo_bat1_sense2
- J405 pad 7: /lipo_bat1_sense3 -> /Power/lipo_bat1_sense3
- J405 pad 8: /lipo_bat1_sense4 -> /Power/lipo_bat1_sense4
- J405 pad 9: /lipo_bat1_sense5 -> /Power/lipo_bat1_sense5
- J406 pad 5: /Power/3v_measured_BATT+ -> Net-(J406-Pad5)
- J406 pad 6: +BATT -> Net-(J406-Pad6)
- J407 pad 5: /Power/5v_measured_BATT+ -> Net-(J407-Pad5)
- J407 pad 6: +BATT -> Net-(J407-Pad6)
- J501 pad 3: /usb_data_D0 -> /Telemetry/usb_data_D0
- J501 pad 4: /usb_data_D1 -> /Telemetry/usb_data_D1
- J503 pad 1: +5V -> Net-(J503-Pad1)
- J503 pad 2: -BATT -> Net-(J503-Pad2)
- Q301 pad 1: /Pump/solenoid_mosfet_gate -> /solenoid_mosfet_gate
- R301 pad 2: /Pump/solenoid_mosfet_gate -> /solenoid_mosfet_gate
- TP201 pad 1: Net-(J206-Pad4) -> (no net)
- TP202 pad 1: /leak_sense_output -> (no net)
- U101 pad 18: Net-(U101-Pad18) -> /irid_RXD
- U101 pad 19: Net-(U101-Pad19) -> /irid_TXD
- U101 pad 4: Net-(U101-Pad4) -> /turbine_2_pwm
- U101 pad 47: Net-(U101-Pad47) -> /irid_CTS
- U101 pad 48: Net-(U101-Pad48) -> /irid_RTS
- U101 pad 49: Net-(U101-Pad49) -> /irid_SLEEP
- U101 pad 50: Net-(U101-Pad50) -> /irid_NET_AV
- U101 pad 8: Net-(U101-Pad8) -> /turbine_1_pwm
- U402 pad 1: /3v_measured_BATT+ -> +BATT
- U402 pad 3: +3V3 -> Net-(J406-Pad6)
- U403 pad 1: /5v_measured_BATT+ -> +BATT
- U403 pad 3: +5V -> Net-(J407-Pad6)

Commit message: shortend pcb, ready to route
ready to route, shortend pcb, layout complete
Parts:
- removed H5, H6: MountingHole, MountingHole:MountingHole_5.3mm_M5_Pad
- removed J503: RockBLOCK 9603, Connector_PinSocket_2.54mm:PinSocket_1x10_P2.54mm_Vertical
- removed TP101: i2c_sda_1, TestPoint:TestPoint_Loop_D2.60mm_Drill1.6mm_Beaded
- removed TP102: i2c_scl_1, TestPoint:TestPoint_Loop_D2.60mm_Drill1.6mm_Beaded
- removed TP201: TP_RawLeak, TestPoint:TestPoint_Loop_D2.60mm_Drill1.6mm_Beaded
- removed TP202: TP_LeakSense, TestPoint:TestPoint_Loop_D2.60mm_Drill1.6mm_Beaded
- removed TP301: TP_SolGate, TestPoint:TestPoint_Loop_D2.60mm_Drill1.6mm_Beaded
- removed TP302: TP_SolVolt, TestPoint:TestPoint_Loop_D2.60mm_Drill1.6mm_Beaded
- removed TP304: TP_SolBat+, TestPoint:TestPoint_Loop_D2.60mm_Drill1.6mm_Beaded
- moved J204 242.2 mm to (311.9, 139.4), turned to 270 degrees
- moved J205 238.3 mm to (311.7, 160.5), turned to 270 degrees
- moved D301 222.9 mm to (312.7, 92.5), turned to 180 degrees
- moved R102 160.7 mm to (164.6, 162.1)
- moved R101 139.6 mm to (164.6, 156.7)
- moved Q301 134.5 mm to (301.0, 104.1), turned to 90 degrees
- moved J101 123.6 mm to (175.3, 114.0), turned to 90 degrees
- moved U402 118.7 mm to (73.7, 134.9), turned to 90 degrees
- moved U403 118.3 mm to (73.4, 121.4), turned to 90 degrees
- moved U102 113.3 mm to (220.5, 133.3)
- moved J208 104.4 mm to (128.3, 138.9), turned to 270 degrees
- moved U202 93.3 mm to (183.4, 131.6)
- moved BT101 92.7 mm to (156.2, 135.4)
- moved J405 91.6 mm to (90.2, 99.1), turned to 0 degrees
- moved R301 82.9 mm to (260.1, 134.9)
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Connections:
- J501 pad 3: /Telemetry/usb_data_D0 -> /usb_data_D0
- J501 pad 4: /Telemetry/usb_data_D1 -> /usb_data_D1
Other:
- board size 304.1 x 76.2 mm -> 261.4 x 76.2 mm
- net class power: trace_width 0.75 -> 1

Commit message: ready for layout
- added batt solder tabs
- swapped some terminal blocks with microfit connectors
- shortened board, tightened layout
- tried to space everything out properly
Parts:
- added J302: VL6180 Range Sensor, Connector_Molex:Molex_Micro-Fit_3.0_43045-0421_2x02-1MP_P3.00mm_Horizontal, F.Cu at (210.8, 98.8)
- added J408: BATT+, TestPoint:TestPoint_Pad_4.0x4.0mm, F.Cu at (163.7, 91.4)
- added U201: QuickFit_02x03_Header-Connector, Connector_Molex:Molex_Micro-Fit_3.0_43045-0621_2x03-1MP_P3.00mm_Horizontal, F.Cu at (63.8, 151.9)
- J201, J202: footprint TerminalBlock_CUI:CUI_TBP01R1W-508-04BE -> Connector_Molex:Molex_Micro-Fit_3.0_43045-0421_2x02-1MP_P3.00mm_Horizontal
- J401: footprint Connector_Molex:Molex_Micro-Fit_3.0_43045-1600_2x08_P3.00mm_Horizontal -> Connector_Molex:Molex_Micro-Fit_3.0_43045-1621_2x08-1MP_P3.00mm_Horizontal
- J404: value Switch Bulkhead -> BATT-; footprint TerminalBlock_CUI:CUI_TBP01R1W-508-02BE -> TestPoint:TestPoint_Pad_4.0x4.0mm
- moved J404 112.5 mm to (157.7, 91.4), turned to 0 degrees
- moved J402 101.9 mm to (222.2, 93.0)
- moved U402 94.9 mm to (166.9, 117.1), turned to 0 degrees
- moved U403 87.4 mm to (159.3, 104.9), turned to 0 degrees
- moved Q301 65.0 mm to (236.0, 104.1), turned to 180 degrees
- moved J203 63.0 mm to (226.8, 111.5)
- moved R201 25.4 mm to (184.4, 117.3), turned to 180 degrees
- moved R202 25.1 mm to (193.0, 117.6), turned to 180 degrees
- moved J202 23.1 mm to (196.6, 98.8)
- moved J502 16.8 mm to (135.4, 111.5), turned to 0 degrees
- moved J303 11.1 mm to (75.9, 118.9)
- moved J101 9.62 mm to (184.7, 112.0)
- moved J304 7.88 mm to (150.9, 122.7)
- moved J308 5.85 mm to (86.1, 111.3)
- moved J307 4.58 mm to (95.8, 111.3)
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Connections:
- net /3v3_feather renamed Net-(U102-Pad15)
- J404 pad 1: /Power/external_switch_A -> /Power/raw_BATT-
- SW401 pad 2: /Power/external_switch_B -> /ext_sw_B
- SW401 pad 3: /Power/external_switch_A -> /ext_sw_A
- U101 pad 87: (no net) -> Net-(R101-Pad2)
- U101 pad 88: (no net) -> Net-(R102-Pad2)
- U401 pad 5: /Power/external_switch_A -> /ext_sw_A
- U401 pad 6: /Power/external_switch_B -> /ext_sw_B
Other:
- board text added: "J201+J202 1: 5V. 2: GND 3: SCL 4: SDA"
- board text added: "J401 8: RS_RX 16: BAT_TH2 7: RS_TX 15: BAT_TH1 6: USB_D1 14: BAT_S1 5: USB_D0 13: BAT_S2 4: USB_5V 12: BAT_S3 3: GND 11: BAT_S4 2: -BAT 10: BAT_S5 1: +BAT 9: RS_GND"
- board text added: "U201 1: 3.3v 2: GND 3: SWA 4: E_SWA 5: E_SWB 6: SDA 7: SCL"

Commit message: ready for routing
- figured out battery input - going with solder strips + sense wires to reduce connector count
Parts:
- removed J405: Battery Input, TerminalBlock_CUI:CUI_TBP01R1W-508-12BE
- removed J501: Serial Telemetry, TerminalBlock_CUI:CUI_TBP01R1W-508-04BE
- added J209: EXT Pressure Sensor, Connector_Molex:Molex_Micro-Fit_3.0_43045-0421_2x02-1MP_P3.00mm_Horizontal, F.Cu at (157.7, 98.8)
- added J409: RAW_BATT-, TestPoint:TestPoint_Pad_4.0x4.0mm, F.Cu at (110.5, 96.9)
- added J410: RAW_BATT+, TestPoint:TestPoint_Pad_4.0x4.0mm, F.Cu at (116.5, 96.9)
- added J411: RAW_BATT-, TestPoint:TestPoint_Plated_Hole_D3.0mm, F.Cu at (110.5, 102.9)
- added J412: RAW_BATT+, TestPoint:TestPoint_Plated_Hole_D3.0mm, F.Cu at (116.5, 102.9)
- added J413: Batt_Therm, Connector_Wire:SolderWire-0.5sqmm_1x02_P4.6mm_D0.9mm_OD2.1mm_Relief, F.Cu at (131.6, 105.2)
- added J414: Batt Sense, Connector_Wire:SolderWire-0.5sqmm_1x05_P4.6mm_D0.9mm_OD2.1mm_Relief, F.Cu at (100.6, 104.6)
- J1: value MAXON Pump Controller -> Pump Controller
- J404: value BATT- -> RAW_BATT-
- J408: value BATT+ -> RAW_BATT+
- moved J205 184.2 mm to (138.9, 96.5), turned to 0 degrees
- moved J204 168.4 mm to (149.1, 96.5), turned to 0 degrees
- moved R102 52.3 mm to (120.4, 134.1)
- moved J408 47.2 mm to (116.5, 91.9)
- moved J404 47.2 mm to (110.4, 91.9)
- moved R101 41.1 mm to (130.3, 134.1)
- moved J301 23.1 mm to (63.8, 159.3)
- moved SW401 22.2 mm to (77.0, 139.7), turned to 270 degrees
- moved U201 19.8 mm to (63.8, 132.1)
- moved BT101 10.7 mm to (149.9, 144.0)
- moved U402 10.00 mm to (162.3, 126.0)
- moved U403 8.92 mm to (162.3, 113.3)
- moved J306 6.10 mm to (129.3, 155.2)
- moved J303 1.80 mm to (75.7, 117.1)
- moved U401 1.52 mm to (86.1, 147.1)
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Connections:
- J401 pad 2: -BATT -> +BATT
- J401 pad 4: /Power/usb_pwr -> -BATT
- J401 pad 5: /Power/usb_data_D0 -> /usb_data_D0
- J401 pad 6: /Power/usb_data_D1 -> /usb_data_D1
- J401 pad 7: /Power/rs232_tx -> /rs232_tx
- J401 pad 8: /Power/rs232_rx -> /rs232_rx
- J401 pad 9: /Power/rs232_gnd -> -BATT
- U101 pad 2: Net-(U101-Pad2) -> /rs232_rx
- U101 pad 3: Net-(U101-Pad3) -> /rs232_tx
- U201 pad 3: /Sensors/ext_SWA -> /ext_sw_A
- U201 pad 4: /i2c_scl_1 -> /ext_sw_B
- U201 pad 6: /Sensors/ext_SWB -> /i2c_scl_1
Other:
- net class hipower added: clearance 0.2, trace_width 3, via_dia 0.8, via_drill 0.4
- net class power: trace_width 1 -> 1.2
- board text added: "U201 1: 3.3v 2: GND 3: E_SWA 4: E_SWB 5: SDA 6: SCL"
- board text removed: "U201 1: 3.3v 2: GND 3: SWA 4: E_SWA 5: E_SWB 6: SDA 7: SCL"
