File: engine-board/engine-board.kicad_pcb (KiCad board)
At the start: 2 copper layers, 261.4 x 76.2 mm, 63 parts, among them J1 Pump Controller, J101 SD Card, J201 Reservoir Pressure Sensor, J202 Bladder Pressure Sensor, J203 HMC6343 COMPASS, J204 QWIIC 1, J205 QWIIC 2, J206 Leak Sensor, J207 BME260 Sensor, J208 RV1805 Clock, J209 EXT Pressure Sensor, J301 Steering Turbines, J302 VL6180 Range Sensor, J303 Pump Current Sensor, J304 VL6180 Range Sensor, J305 Turbine 1 ESC, J306 Turbine 2 ESC, J307 Turbine Current Sensor, J308 Solenoid Current Sensor, J309 Solenoid, J401 USB/SER/CHRGR, J402 Power Rail, J403 Engine Current Sensor, J404 RAW_BATT-, J406 3V Current Sensor, J407 5V Current Sensor, J408 RAW_BATT+, J409 RAW_BATT-, J410 RAW_BATT+, J411 RAW_BATT-, J412 RAW_BATT+, J413 Batt_Therm, J414 Batt Sense, J502 NEO08MU GPS, J504 RockBlock9603, Q301 IRLB8721PBF, SW401 POWER, U101 Teensy3.6_All_Pins, U102 FEATHER_M0_BASIC_PROTO, U201 QuickFit_02x03_Header-Connect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, U202 BN0055 IMU, U401 Pololu_2814, U402 R-78B3.3-2.0, U403 R-78B5.0-2.0

Commit message: Verions 1.0 done + ordered
added routes, submitted order
Parts:
- J209: value EXT Pressure Sensor -> External Pressure Sensor
Connections:
- J413 pad 1: /Power/lipo_bat_therm1 -> /Power/lipo_bat1_therm1
- J413 pad 2: /Power/lipo_bat_therm2 -> /Power/lipo_bat1_therm2
Routing:
- net -BATT: track 0.00 -> 798.7 mm, vias 0 -> 1
- net /i2c_scl_1: track 0.00 -> 506.8 mm
- net /i2c_sda_1: track 0.00 -> 481.5 mm
- net +3V3: track 0.00 -> 450.1 mm, vias 0 -> 4
- net /rs232_tx: track 0.00 -> 259.4 mm
- net /Pump/solenoid_measured_BATT+: track 0.00 -> 255.1 mm
- net /rs232_rx: track 0.00 -> 253.7 mm
- net +5V: track 0.00 -> 251.3 mm, vias 0 -> 2
- net /Pump/pump_measured_BATT+: track 0.00 -> 233.1 mm, vias 0 -> 1
- net /turbine_2_pwm: track 0.00 -> 223.7 mm
- net +BATT: track 0.00 -> 223.0 mm, vias 0 -> 1
- net /Power/switched_BATT+: track 0.00 -> 201.9 mm, vias 0 -> 3
- net /Pump/turbine1_grn: track 0.00 -> 159.2 mm
- net /Pump/turbine1_blu: track 0.00 -> 154.0 mm, vias 0 -> 1
- net /Pump/turbine1_measured_pwr: track 0.00 -> 149.5 mm, vias 0 -> 2
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Other:
- net class hipower: trace_width 3 -> 2
- board text added: "SeaFlight Glider 123-1001 V1.0"

Commit message: board smaller
PCB V0.1 Errata:

- [QUESTION: - it looks like 12 on website] polulu 2814 has 16 pin footprint instead of 12...  AAACK!!!
- 5v and 3.3v traces could be wider
- [FIXED] fail: going into the power schematic scl + sda are swapped...
- [FIXED - moved to miniofit] pump controller silkscreen is wrong
- [FIXED] NOTE: just switch ALL to the minifit??
- [FIXED - will be on top, but not needed now] ADD: Ethernet connection from the teensy to the host computer board.
- [FIXED - going to use Qwiic) 9 Axis Mopak: wrong footprint - holes too small, spacing seems good, create outline as it bumps into feather header
- [FIXED] RV1805:  power + GND swapped... and I can’t seem to find them.
- [FIXED] 2 pressure sensors, the same i2c address... rerouted to 2nd i2c port on teensy
- [NOT NEEDED - adding display] Add RGB LED... it will be helpful for debugging.
- [FIXED - kindof - moved to micro-fit, might need to wire this directly to bulkhead] Turbine ferrules for power are 12 gauge - need bigger screw terminals if that is the connection method
- [FIXED] Feather footprint - lookup exactly what feather boards need for support..
- [FIXED] pump_motor_pwm is not connected to the TEENSY!!  blerg.  (jumper to pin 13 of feather for now)
- [FIXED - added FET] Maxon 70/30 POWER?  Think about power FET or ‘sleep’ to turn it off.
- [FIXED - added to bulkhead connector] Teensy 4.1 Program + ON/OFF pins - research how to extend these
- [TODO] remove VL6180 range sensor
- [LATER - will add to cost.. possibly remove?] put battery on back side
- add silkscreen for polulu
- [FIXED] Reorganize connectors:
    - Pump motor connectors go on end - attached in closing
    - bulkhead connectors go on side as they will always be attached
Parts:
- removed J101: SD Card, Connector_PinSocket_2.54mm:PinSocket_1x08_P2.54mm_Vertical
- removed J502: NEO08MU GPS, Connector_PinSocket_2.54mm:PinSocket_1x08_P2.54mm_Vertical
- removed J504: RockBlock9603, Connector_PinSocket_2.54mm:PinSocket_1x10_P2.54mm_Vertical
- removed JP101, JP102, JP201: PumpAngGND, Jumper:SolderJumper-2_P1.3mm_Open_Pad1.0x1.5mm
- removed JP103: pump_pwm1, Jumper:SolderJumper-2_P1.3mm_Open_Pad1.0x1.5mm
- removed JP104: pump_pwm2, Jumper:SolderJumper-2_P1.3mm_Open_Pad1.0x1.5mm
- removed U201: QuickFit_02x03_Header-Connector, Connector_Molex:Molex_Micro-Fit_3.0_43045-0621_2x03-1MP_P3.00mm_Horizontal
- removed U202: BN0055 IMU, Sensor_Motion:ADA_BN0055
- removed U401: Pololu_2814, Module:Pololu_Breakout-16_15.2x20.3mm
- added J310: QWIIC 4, Connector_JST:JST_SH_BM04B-SRSS-TB_1x04-1MP_P1.00mm_Vertical, F.Cu at (73.0, 92.1)
- added J311: QWIIC 3, Connector_JST:JST_SH_BM04B-SRSS-TB_1x04-1MP_P1.00mm_Vertical, F.Cu at (226.1, 92.7)
- added J415: Telemetry Bottle, Connector_Molex:Molex_Micro-Fit_3.0_43045-1621_2x08-1MP_P3.00mm_Horizontal, F.Cu at (114.0, 98.5)
- added J416: Telemetry Current Sensor, Connector_PinSocket_2.54mm:PinSocket_1x08_P2.54mm_Vertical, F.Cu at (131.4, 111.1)
- added J501: Solenoid, Connector_Molex:Molex_Micro-Fit_3.0_43045-0221_2x01-1MP_P3.00mm_Horizontal, F.Cu at (63.5, 112.4)
- added J503: RockBLOCK 9603, Connector_PinSocket_2.54mm:PinSocket_1x10_P2.54mm_Vertical, F.Cu at (197.5, 109.9)
- added Q401: IRLB8721PBF, Package_TO_SOT_THT:TO-220-3_Vertical, F.Cu at (156.8, 121.6)
- added Q501: IRLB8721PBF, Package_TO_SOT_THT:TO-220-3_Vertical, F.Cu at (89.5, 137.5)
- added R401: 10kohm, Resistor_THT:R_Axial_DIN0204_L3.6mm_D1.6mm_P5.08mm_Vertical, F.Cu at (158.8, 127.6)
- added R501: 10kohm, Resistor_THT:R_Axial_DIN0204_L3.6mm_D1.6mm_P5.08mm_Vertical, F.Cu at (80.1, 132.7)
- J1: footprint TerminalBlock_CUI:CUI_TBP01R1W-508-12BE -> Connector_Molex:Molex_Micro-Fit_3.0_43045-1221_2x06-1MP_P3.00mm_Horizontal
- J201: footprint Connector_Molex:Molex_Micro-Fit_3.0_43045-0421_2x02-1MP_P3.00mm_Horizontal -> Connector_Molex:Molex_Micro-Fit_3.0_43650-0400_1x04_P3.00mm_Horizontal
- J203: footprint Connector_PinSocket_2.54mm:PinSocket_1x04_P2.54mm_Vertical -> Connector_Molex:Molex_Micro-Fit_3.0_43045-0421_2x02-1MP_P3.00mm_Horizontal
- J206: footprint TerminalBlock_CUI:CUI_TBP01R1W-508-04BE -> Connector_Molex:Molex_Micro-Fit_3.0_43045-0421_2x02-1MP_P3.00mm_Horizontal
- J304: value VL6180 Range Sensor -> Conn_02x03_Top_Bottom; footprint Connector_PinSocket_2.54mm:PinSocket_1x06_P2.54mm_Vertical -> Connector_Molex:Molex_Micro-Fit_3.0_43045-0621_2x03-1MP_P3.00mm_Horizontal
- J305, J306: footprint TerminalBlock_CUI:CUI_TBP01R1W-508-08BE -> Connector_Molex:Molex_Micro-Fit_3.0_43045-0821_2x04-1MP_P3.00mm_Horizontal
- J309: value Solenoid -> BME280; footprint TerminalBlock_CUI:CUI_TBP01R1W-508-02BE -> Connector_PinSocket_2.54mm:PinSocket_1x04_P2.54mm_Vertical
- moved J1 231.7 mm to (63.5, 148.5), turned to 90 degrees
- moved D301 212.1 mm to (101.6, 134.0), turned to 0 degrees
- moved J206 172.7 mm to (87.9, 155.5), turned to 180 degrees
- moved J302 159.6 mm to (63.5, 160.2), turned to 90 degrees
- moved J309 138.3 mm to (146.0, 118.7), turned to 180 degrees
- moved Q301 136.7 mm to (104.8, 142.6), turned to 0 degrees
- moved J202 135.5 mm to (63.5, 124.7), turned to 90 degrees
- moved J402 134.4 mm to (99.1, 146.7), turned to -90 degrees
- moved J201 121.0 mm to (63.5, 103.5), turned to 90 degrees
- moved J414 100.7 mm to (201.3, 104.3)
- moved J204 99.3 mm to (224.2, 161.5), turned to 180 degrees
- moved J408 98.9 mm to (215.4, 91.6)
- moved J409 98.9 mm to (209.4, 96.5)
- moved J411 98.9 mm to (209.4, 102.5)
- moved J404 98.9 mm to (209.4, 91.6)
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Connections:
- J1 pad 3: -BATT -> Net-(J1-Pad3)
- J1 pad 4: -BATT -> Net-(J1-Pad3)
- J201 pad 3: /i2c_scl_1 -> /i2c_scl_2
- J201 pad 4: /i2c_sda_1 -> /i2c_sda_2
- J206 pad 3: Net-(J206-Pad3) -> unconnected-(J206-Pad3)
- J208 pad 1: +3V3 -> -BATT
- J208 pad 2: -BATT -> +3V3
- J303 pad 5: Net-(J303-Pad5) -> unconnected-(J303-Pad5)
- J304 pad 1: Net-(J304-Pad1) -> +3V3
- J304 pad 2: Net-(J304-Pad2) -> -BATT
- J304 pad 3: /i2c_scl_1 -> /ext_sw_A
- J304 pad 4: /i2c_sda_1 -> /i2c_scl_1
- J304 pad 5: +3V3 -> /i2c_sda_1
- J304 pad 6: -BATT -> /ext_sw_B
- J305 pad 5: Net-(J305-Pad5) -> unconnected-(J305-Pad5)
- J306 pad 5: Net-(J306-Pad5) -> unconnected-(J306-Pad5)
- J307 pad 5: Net-(J307-Pad5) -> unconnected-(J307-Pad5)
- J308 pad 5: Net-(J308-Pad5) -> unconnected-(J308-Pad5)
- J309 pad 1: Net-(D301-Pad2) -> -BATT
- J309 pad 2: /Pump/solenoid_measured_BATT+ -> +3V3
- J401 pad 15: /Power/lipo_bat1_therm1 -> /TEENSY_PROGRAM
- J401 pad 16: /Power/lipo_bat1_therm2 -> GND
- J402 pad 4: /i2c_sda_1 -> /i2c_scl_1
- J402 pad 5: /i2c_scl_1 -> /i2c_sda_1
- J403 pad 3: /i2c_sda_1 -> /i2c_scl_1
- J403 pad 4: /i2c_scl_1 -> /i2c_sda_1
- J403 pad 5: Net-(J403-Pad5) -> unconnected-(J403-Pad5)
- J406 pad 3: /i2c_sda_1 -> /i2c_scl_1
- J406 pad 4: /i2c_scl_1 -> /i2c_sda_1
- J406 pad 5: Net-(J406-Pad5) -> unconnected-(J406-Pad5)
- J407 pad 3: /i2c_sda_1 -> /i2c_scl_1
- J407 pad 4: /i2c_scl_1 -> /i2c_sda_1
- J407 pad 5: Net-(J407-Pad5) -> unconnected-(J407-Pad5)
- SW401 pad 1: Net-(SW401-Pad1) -> unconnected-(SW401-Pad1)
- U101 pad 10: Net-(U101-Pad10) -> unconnected-(U101-Pad10)
- U101 pad 11: Net-(U101-Pad11) -> unconnected-(U101-Pad11)
- U101 pad 12: Net-(U101-Pad12) -> unconnected-(U101-Pad12)
- U101 pad 13: Net-(U101-Pad13) -> unconnected-(U101-Pad13)
- U101 pad 14: Net-(U101-Pad14) -> unconnected-(U101-Pad14)
- U101 pad 16: Net-(U101-Pad16) -> unconnected-(U101-Pad16)
- U101 pad 17: Net-(U101-Pad17) -> unconnected-(U101-Pad17)
- U101 pad 21: Net-(U101-Pad21) -> /pump_motor_pwm
- U101 pad 22: Net-(U101-Pad22) -> /pumpPower_mosfet_gate
- U101 pad 23: Net-(U101-Pad23) -> unconnected-(U101-Pad23)
- U101 pad 24: Net-(U101-Pad24) -> unconnected-(U101-Pad24)
- U101 pad 28: Net-(U101-Pad28) -> /TEENSY_PROGRAM
- U101 pad 29: Net-(U101-Pad29) -> unconnected-(U101-Pad29)
- U101 pad 30: Net-(U101-Pad30) -> /btn_4
- U101 pad 31: Net-(U101-Pad31) -> /btn_3
- U101 pad 34: Net-(U101-Pad34) -> /i2c_scl_2
- U101 pad 35: Net-(U101-Pad35) -> /i2c_sda_2
- U101 pad 36: Net-(U101-Pad36) -> /gps_pss
- U101 pad 37: Net-(U101-Pad37) -> /btn_2
- U101 pad 38: Net-(U101-Pad38) -> /btn_1
- U101 pad 40: Net-(U101-Pad40) -> unconnected-(U101-Pad40)
- U101 pad 5: Net-(U101-Pad5) -> unconnected-(U101-Pad5)
- U101 pad 51: Net-(JP101-Pad1) -> unconnected-(U101-Pad51)
- U101 pad 52: Net-(U101-Pad52) -> unconnected-(U101-Pad52)
- U101 pad 53: Net-(U101-Pad53) -> unconnected-(U101-Pad53)
- U101 pad 54: Net-(U101-Pad54) -> unconnected-(U101-Pad54)
- U101 pad 57: Net-(U101-Pad57) -> unconnected-(U101-Pad57)
- U101 pad 58: Net-(U101-Pad58) -> unconnected-(U101-Pad58)
- U101 pad 59: Net-(U101-Pad59) -> unconnected-(U101-Pad59)
- U101 pad 6: Net-(U101-Pad6) -> unconnected-(U101-Pad6)
- U101 pad 60: Net-(U101-Pad60) -> unconnected-(U101-Pad60)
- U101 pad 7: Net-(U101-Pad7) -> unconnected-(U101-Pad7)
- U101 pad 9: Net-(U101-Pad9) -> unconnected-(U101-Pad9)
- U102 pad 1: Net-(U102-Pad1) -> unconnected-(U102-Pad1)
- U102 pad 10: /pump_motor_analog_current -> unconnected-(U102-Pad10)
- U102 pad 11: /pump_motor_analog_speed -> unconnected-(U102-Pad11)
- U102 pad 12: Net-(U102-Pad12) -> unconnected-(U102-Pad12)
- U102 pad 14: Net-(JP102-Pad2) -> unconnected-(U102-Pad14)
- U102 pad 15: Net-(U102-Pad15) -> +3V3
- U102 pad 16: Net-(U102-Pad16) -> /btn_4
- U102 pad 17: Net-(U102-Pad17) -> unconnected-(U102-Pad17)
- U102 pad 18: Net-(U102-Pad18) -> unconnected-(U102-Pad18)
- U102 pad 19: +5V -> unconnected-(U102-Pad19)
- U102 pad 2: Net-(R102-Pad2) -> unconnected-(U102-Pad2)
- U102 pad 20: Net-(JP103-Pad1) -> unconnected-(U102-Pad20)
- U102 pad 21: /pump_motor_ccw -> unconnected-(U102-Pad21)
- U102 pad 22: /pump_motor_cw -> unconnected-(U102-Pad22)
- U102 pad 23: Net-(JP104-Pad1) -> unconnected-(U102-Pad23)
- U102 pad 24: /turbine_1_pwm -> /btn_3
- U102 pad 25: /turbine_2_pwm -> /btn_2
- U102 pad 26: /imu_cs -> /btn_1
- U102 pad 3: Net-(R101-Pad2) -> unconnected-(U102-Pad3)
- U102 pad 4: /SDO -> unconnected-(U102-Pad4)
- U102 pad 5: /SDI -> unconnected-(U102-Pad5)
- U102 pad 6: /SCK -> unconnected-(U102-Pad6)
- U102 pad 7: /sdcard_cs -> unconnected-(U102-Pad7)
- U102 pad 8: /leak_sense_output -> unconnected-(U102-Pad8)
- U102 pad 9: /solenoid_mosfet_gate -> unconnected-(U102-Pad9)
Routing:
- net -BATT: track 798.7 -> 0.00 mm, vias 1 -> 0
- net /i2c_scl_1: track 506.8 -> 0.00 mm
- net /i2c_sda_1: track 481.5 -> 0.00 mm
- net +3V3: track 450.1 -> 0.00 mm, vias 4 -> 0
- net /rs232_tx: track 259.4 -> 0.00 mm
- net /Pump/solenoid_measured_BATT+: track 255.1 -> 0.00 mm
- net /rs232_rx: track 253.7 -> 0.00 mm
- net +5V: track 251.3 -> 0.00 mm, vias 2 -> 0
- net /Pump/pump_measured_BATT+: track 233.1 -> 0.00 mm, vias 1 -> 0
- net /turbine_2_pwm: track 223.7 -> 0.00 mm
- net +BATT: track 223.0 -> 0.00 mm, vias 1 -> 0
- net /Power/switched_BATT+: track 201.9 -> 0.00 mm, vias 3 -> 0
- net /Pump/turbine1_grn: track 159.2 -> 0.00 mm
- net /Pump/turbine1_blu: track 154.0 -> 0.00 mm, vias 1 -> 0
- net /Pump/turbine1_measured_pwr: track 149.5 -> 0.00 mm, vias 2 -> 0
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Other:
- board size 261.4 x 76.2 mm -> 181.6 x 76.2 mm
- net class Default removed
- net class hipower removed
- net class power removed
- board text added: "SeaFlight Glider 123-1001 V1.1"
- board text added: "SeaFlight Glider V1.2"
- board text removed: "J201+J202 1: 5V. 2: GND 3: SCL 4: SDA"
- board text removed: "J401 8: RS_RX 16: BAT_TH2 7: RS_TX 15: BAT_TH1 6: USB_D1 14: BAT_S1 5: USB_D0 13: BAT_S2 4: USB_5V 12: BAT_S3 3: GND 11: BAT_S4 2: -BAT 10: BAT_S5 1: +BAT 9: RS_GND"
- board text removed: "SeaFlight Glider 123-1001 V1.0"
