File: engine-board/engine-board.sch (KiCad schematic (older format))
At the start: 31 parts, among them J10 USB/SER/CHRGR, J11 Engine Current Sensor, J12 Micro-Fit_2x04, J20 POWER_JACK, J21 73099-0, J22 73099-0, J24 Battery Input, J25 Turbine ESC, J27 Leak Detector, J28 Maxon Motor, J31 Solenoid, J32 Solenoid Current Sensor, J33 BME280 Sensor, J34 RV1805 Clock, J35 Reservoir Pressure Sensor, J36 Bladder Pressure Sensor, J37 VL6180 Range Sensor, J42 HMC6343 COMPASS, J43 NEO08MU GPS, J44 Turbine Current Sensor, Q1 IRLB8721PBF, U1 FEATHER_M0_BASIC_PROTO, U2 R-78B5.0-2.0, U3 R-78B3.3-2.0

Commit message: all parts in schematic + pcb
still need to route + add mounting holes based on mechanical design.. ready for initial review
Parts:
- removed J20: POWER_JACK, Connector_BarrelJack:BarrelJack_CUI_PJ-063AH_Horizontal, symbol engine-board-rescue:POWER_JACK-SparkFun-Connectors
- removed J21, J22: 73099-0, Connector:Banana_Jack_1Pin, symbol engine-board-rescue:73099-0-73099-0
- removed J27: Leak Detector, Connector_Molex:Molex_Micro-Fit_3.0_43650-0300_1x03_P3.00mm_Horizontal, symbol Connector:Conn_01x03_Female
- removed J28: Maxon Motor, Connector_Molex:Molex_Micro-Fit_3.0_43045-1610_2x08-1MP_P3.00mm_Horizontal, symbol Connector_Generic:Conn_02x08_Top_Bottom
- removed J31: Solenoid, Connector_Molex:Molex_Micro-Latch_53254-0270_1x02_P2.00mm_Horizontal, symbol Connector:Conn_01x02_Female
- added J1: MAXON Pump Controller, TerminalBlock_CUI:CUI_TBP01R1W-508-12BE, symbol Connector_Generic:Conn_02x06_Top_Bottom
- added J2: Power Rail, Connector_Molex:Molex_KK-254_AE-6410-08A_1x08_P2.54mm_Vertical, symbol Connector:Conn_01x08_Female
- added J27: Reservoir Pressure Sensor, TerminalBlock_CUI:CUI_TBP01R1W-508-04BE, symbol Connector_Generic:Conn_02x02_Top_Bottom
- added J31: Solenoid, TerminalBlock_CUI:CUI_TBP01R1W-508-02BE, symbol SeaFlight~Glider:Solenoid_Socket_2pin
- added J45: Engine Current Sensor, Connector_Molex:Molex_KK-254_AE-6410-06A_1x06_P2.54mm_Vertical, symbol Connector:Conn_01x06_Female
- added J47: QWIIC 1, Connector_Molex:Molex_KK-254_AE-6410-04A_1x04_P2.54mm_Vertical, symbol Connector:Conn_01x04_Female
- added J48: QWIIC 2, Connector_Molex:Molex_KK-254_AE-6410-04A_1x04_P2.54mm_Vertical, symbol Connector:Conn_01x04_Female
- added J50: SD Card, Connector_Molex:Molex_KK-254_AE-6410-08A_1x08_P2.54mm_Vertical, symbol Connector:Conn_01x08_Female
- added JP10: teensy_cw, Jumper:SolderJumper-2_P1.3mm_Open_Pad1.0x1.5mm, symbol Jumper:SolderJumper_2_Open
- added JP11: pump_speed, Jumper:SolderJumper-2_P1.3mm_Open_Pad1.0x1.5mm, symbol Jumper:SolderJumper_2_Open
- added JP12: pump_current, Jumper:SolderJumper-2_P1.3mm_Open_Pad1.0x1.5mm, symbol Jumper:SolderJumper_2_Open
- added JP13: solenoid_gate, Jumper:SolderJumper-2_P1.3mm_Open_Pad1.0x1.5mm, symbol Jumper:SolderJumper_2_Open
- added JP14: leak_in, Jumper:SolderJumper-2_P1.3mm_Open_Pad1.0x1.5mm, symbol Jumper:SolderJumper_2_Open
- added JP15: imu_cs, Jumper:SolderJumper-2_P1.3mm_Open_Pad1.0x1.5mm, symbol Jumper:SolderJumper_2_Open
- added JP5: IMU PS1 Jump, Connector_PinHeader_2.54mm:PinHeader_1x02_P2.54mm_Vertical, symbol Jumper:Jumper_2_Open
- added JP6: IMU PS0 Jump, Connector_PinHeader_2.54mm:PinHeader_1x02_P2.54mm_Vertical, symbol Jumper:Jumper_2_Open
- added JP7: teensy_scl, Jumper:SolderJumper-2_P1.3mm_Open_Pad1.0x1.5mm, symbol Jumper:SolderJumper_2_Open
- added JP8: teensy sda, Jumper:SolderJumper-2_P1.3mm_Open_Pad1.0x1.5mm, symbol Jumper:SolderJumper_2_Open
- added JP9: teensy_ccw, Jumper:SolderJumper-2_P1.3mm_Open_Pad1.0x1.5mm, symbol Jumper:SolderJumper_2_Open
- added R4: 1kohm, Resistor_THT:R_Axial_DIN0204_L3.6mm_D1.6mm_P5.08mm_Vertical, symbol Device:R_Small
- added R5: 2kohm, Resistor_THT:R_Axial_DIN0204_L3.6mm_D1.6mm_P5.08mm_Vertical, symbol Device:R_Small
- added TP1: raw leak, TestPoint:TestPoint_THTPad_3.0x3.0mm_Drill1.5mm, symbol Connector:TestPoint
- added TP2: leak3v3, TestPoint:TestPoint_THTPad_3.0x3.0mm_Drill1.5mm, symbol Connector:TestPoint
- added U4: Teensy4.1, Module:Teensy41, symbol teensy:Teensy4.1
- added U51: IMU_BN0080, Module:DIP-24_900_ELL, symbol Sensor_Motion:IMU_BN0080
- J11: value Engine Current Sensor -> Pump Current Sensor
- J12: value Micro-Fit_2x04 -> Steering Turbines; footprint Connector_Molex:Molex_Micro-Fit_3.0_43045-0621_2x03-1MP_P3.00mm_Horizontal -> TerminalBlock_CUI:CUI_TBP01R1W-508-08BE
- J24: footprint Connector_Molex:Molex_Micro-Fit_3.0_43045-1221_2x06-1MP_P3.00mm_Horizontal -> TerminalBlock_CUI:CUI_TBP01R1W-508-12BE
- J25: footprint Connector_Molex:Molex_Micro-Fit_3.0_43045-1621_2x08-1MP_P3.00mm_Horizontal -> TerminalBlock_CUI:CUI_TBP01R1W-508-08BE
- J35, J36: footprint Connector_Molex:Molex_Micro-Fit_3.0_43045-0410_2x02-1MP_P3.00mm_Horizontal -> TerminalBlock_CUI:CUI_TBP01R1W-508-04BE
- JP50: value SolderJumper -> pump_pwm1
- JP51: value SolderJumper -> pump_pwm2
Connections:
- net labels added: 3v3_feather, SCK, SDI, SDO, imu_cs, pin6_feather, pin7_feather, pump_measured_BATT+, sdcard_cs
- net labels removed: external_12v_gnd, external_12v_plus, usb_gnd
- wire segments 193 -> 296
Other:
- moved on the sheet: J12, U2, U3

Commit message: fixed size, mounting holes
size is 3"x12", mounting holes aligned with engine bracket, added IMU, Teensy, proper turbine PWM/speed control plugs, converted battery + turbine bulkhead connectors to Molex Minifit
Parts:
- added J53: Switch Bulkhead, TerminalBlock_CUI:CUI_TBP01R1W-508-02BE, symbol Connector:Conn_01x02_Female
- added J62: Turbine 2 ESC, TerminalBlock_CUI:CUI_TBP01R1W-508-08BE, symbol Connector_Generic:Conn_02x04_Top_Bottom
- added U10: Pololu_2812, Module:Pololu_SlidePwrSwitch, symbol Regulator_Controller:Pololu_2812
- J10: footprint Connector_PinHeader_2.54mm:CUI_TBP01R1W-508-16BE -> Connector_Molex:Molex_Micro-Fit_3.0_43045-1600_2x08_P3.00mm_Horizontal
- J12: footprint TerminalBlock_CUI:CUI_TBP01R1W-508-08BE -> Connector_Molex:Molex_Micro-Fit_3.0_43045-0821_2x04-1MP_P3.00mm_Horizontal
- J27: value Reservoir Pressure Sensor -> Leak Sensor
- J61: renamed from J25; value Turbine ESC -> Turbine 1 ESC
Connections:
- net labels added: external_switch_A, external_switch_B, raw_BATT+, raw_BATT-, turbine_1_pwm, turbine_2_pwm
- net labels removed: pin6_feather, pin7_feather
- wire segments 296 -> 328
Other:
- moved on the sheet: J11, J12, J2, J24, J43, J44, J45, J61

Commit message: pushed everything to silkscreen from f.fab
almost final..  just needs routing..
Parts:
- JP1: value SolderJumper -> PumpAngGND
Changed lines of the file:
@@
 P 4300 6700
 F 0 "JP1" H 4300 6905 50  0000 C CNN
-F 1 "SolderJumper" H 4300 6814 50  0000 C CNN
+F 1 "PumpAngGND" H 4300 6814 50  0000 C CNN
 F 2 "Jumper:SolderJumper-2_P1.3mm_Open_Pad1.0x1.5mm" H 4300 6700 50  0001 C CNN
 F 3 "~" H 4300 6700 50  0001 C CNN

Commit message: Broke up into multiple schematics
- broke up into multiple schematics
- replaced some parts based on availability of parts
Parts:
- removed D2: 1N4001, Diode_THT:D_DO-41_SOD81_P10.16mm_Horizontal, symbol Diode:1N4001
- removed J1: MAXON Pump Controller, TerminalBlock_CUI:CUI_TBP01R1W-508-12BE, symbol Connector_Generic:Conn_02x06_Top_Bottom
- removed J10: USB/SER/CHRGR, Connector_Molex:Molex_Micro-Fit_3.0_43045-1600_2x08_P3.00mm_Horizontal, symbol Connector:QuickFit_01x16_Header
- removed J11: Pump Current Sensor, Connector_Molex:Molex_KK-254_AE-6410-06A_1x06_P2.54mm_Vertical, symbol Connector:Conn_01x06_Female
- removed J12: Steering Turbines, Connector_Molex:Molex_Micro-Fit_3.0_43045-0821_2x04-1MP_P3.00mm_Horizontal, symbol Connector_Generic:Conn_02x04_Top_Bottom
- removed J2: Power Rail, Connector_Molex:Molex_KK-254_AE-6410-08A_1x08_P2.54mm_Vertical, symbol Connector:Conn_01x08_Female
- removed J24: Battery Input, TerminalBlock_CUI:CUI_TBP01R1W-508-12BE, symbol Connector_Generic:Conn_02x06_Top_Bottom
- removed J27: Leak Sensor, TerminalBlock_CUI:CUI_TBP01R1W-508-04BE, symbol Connector_Generic:Conn_02x02_Top_Bottom
- removed J31: Solenoid, TerminalBlock_CUI:CUI_TBP01R1W-508-02BE, symbol SeaFlight~Glider:Solenoid_Socket_2pin
- removed J32: Solenoid Current Sensor, Connector_Molex:Molex_KK-254_AE-6410-06A_1x06_P2.54mm_Vertical, symbol Connector:Conn_01x06_Female
- removed J33: BME280 Sensor, Connector_Molex:Molex_KK-254_AE-6410-06A_1x06_P2.54mm_Vertical, symbol Connector:Conn_01x06_Female
- removed J34: RV1805 Clock, Connector_Molex:Molex_KK-254_AE-6410-07A_1x07_P2.54mm_Vertical, symbol Connector:Conn_01x07_Female
- removed J35: Reservoir Pressure Sensor, TerminalBlock_CUI:CUI_TBP01R1W-508-04BE, symbol Connector_Generic:Conn_02x02_Top_Bottom
- removed J36: Bladder Pressure Sensor, TerminalBlock_CUI:CUI_TBP01R1W-508-04BE, symbol Connector_Generic:Conn_02x02_Top_Bottom
- removed J37: VL6180 Range Sensor, Connector_Molex:Molex_KK-254_AE-6410-06A_1x06_P2.54mm_Vertical, symbol Connector:Conn_01x06_Female
- removed J42: HMC6343 COMPASS, Connector_Molex:Molex_KK-254_AE-6410-04A_1x04_P2.54mm_Vertical, symbol Connector:Conn_01x04_Female
- removed J43: NEO08MU GPS, Connector_Molex:Molex_KK-254_AE-6410-08A_1x08_P2.54mm_Vertical, symbol Connector:Conn_01x08_Female
- removed J44: Turbine Current Sensor, Connector_Molex:Molex_KK-254_AE-6410-06A_1x06_P2.54mm_Vertical, symbol Connector:Conn_01x06_Female
- removed J45: Engine Current Sensor, Connector_Molex:Molex_KK-254_AE-6410-06A_1x06_P2.54mm_Vertical, symbol Connector:Conn_01x06_Female
- removed J47: QWIIC 1, Connector_Molex:Molex_KK-254_AE-6410-04A_1x04_P2.54mm_Vertical, symbol Connector:Conn_01x04_Female
- removed J48: QWIIC 2, Connector_Molex:Molex_KK-254_AE-6410-04A_1x04_P2.54mm_Vertical, symbol Connector:Conn_01x04_Female
- removed J50: SD Card, Connector_Molex:Molex_KK-254_AE-6410-08A_1x08_P2.54mm_Vertical, symbol Connector:Conn_01x08_Female
- removed J53: Switch Bulkhead, TerminalBlock_CUI:CUI_TBP01R1W-508-02BE, symbol Connector:Conn_01x02_Female
- removed J61: Turbine 1 ESC, TerminalBlock_CUI:CUI_TBP01R1W-508-08BE, symbol Connector_Generic:Conn_02x04_Top_Bottom
- removed J62: Turbine 2 ESC, TerminalBlock_CUI:CUI_TBP01R1W-508-08BE, symbol Connector_Generic:Conn_02x04_Top_Bottom
- removed JP10: teensy_cw, Jumper:SolderJumper-2_P1.3mm_Open_Pad1.0x1.5mm, symbol Jumper:SolderJumper_2_Open
- removed JP11: pump_speed, Jumper:SolderJumper-2_P1.3mm_Open_Pad1.0x1.5mm, symbol Jumper:SolderJumper_2_Open
- removed JP12: pump_current, Jumper:SolderJumper-2_P1.3mm_Open_Pad1.0x1.5mm, symbol Jumper:SolderJumper_2_Open
- removed JP13: solenoid_gate, Jumper:SolderJumper-2_P1.3mm_Open_Pad1.0x1.5mm, symbol Jumper:SolderJumper_2_Open
- removed JP14: leak_in, Jumper:SolderJumper-2_P1.3mm_Open_Pad1.0x1.5mm, symbol Jumper:SolderJumper_2_Open
- removed JP15: imu_cs, Jumper:SolderJumper-2_P1.3mm_Open_Pad1.0x1.5mm, symbol Jumper:SolderJumper_2_Open
- removed JP5: IMU PS1 Jump, Connector_PinHeader_2.54mm:PinHeader_1x02_P2.54mm_Vertical, symbol Jumper:Jumper_2_Open
- removed JP6: IMU PS0 Jump, Connector_PinHeader_2.54mm:PinHeader_1x02_P2.54mm_Vertical, symbol Jumper:Jumper_2_Open
- removed JP7: teensy_scl, Jumper:SolderJumper-2_P1.3mm_Open_Pad1.0x1.5mm, symbol Jumper:SolderJumper_2_Open
- removed JP8: teensy sda, Jumper:SolderJumper-2_P1.3mm_Open_Pad1.0x1.5mm, symbol Jumper:SolderJumper_2_Open
- removed JP9: teensy_ccw, Jumper:SolderJumper-2_P1.3mm_Open_Pad1.0x1.5mm, symbol Jumper:SolderJumper_2_Open
- removed Q1: IRLB8721PBF, Package_TO_SOT_THT:TO-220-3_Vertical, symbol Transistor_FET:IRLB8721PBF
- removed R3: 10kohm, Resistor_THT:R_Axial_DIN0204_L3.6mm_D1.6mm_P5.08mm_Vertical, symbol Device:R_Small
- removed R4: 1kohm, Resistor_THT:R_Axial_DIN0204_L3.6mm_D1.6mm_P5.08mm_Vertical, symbol Device:R_Small
- removed R5: 2kohm, Resistor_THT:R_Axial_DIN0204_L3.6mm_D1.6mm_P5.08mm_Vertical, symbol Device:R_Small
- removed TP1: raw leak, TestPoint:TestPoint_THTPad_3.0x3.0mm_Drill1.5mm, symbol Connector:TestPoint
- removed TP2: leak3v3, TestPoint:TestPoint_THTPad_3.0x3.0mm_Drill1.5mm, symbol Connector:TestPoint
- removed U10: Pololu_2812, Module:Pololu_SlidePwrSwitch, symbol Regulator_Controller:Pololu_2812
- removed U2: R-78B5.0-2.0, Converter_DCDC:Converter_DCDC_RECOM_R-78B-2.0_THT, symbol Regulator_Switching:R-78B5.0-2.0
- removed U3: R-78B3.3-2.0, Converter_DCDC:Converter_DCDC_RECOM_R-78B-2.0_THT, symbol Regulator_Switching:R-78B3.3-2.0
- removed U4: Teensy4.1, Module:Teensy41, symbol teensy:Teensy4.1
- removed U51: IMU_BN0080, Module:DIP-24_900_ELL, symbol Sensor_Motion:IMU_BN0080
- added BT101: Battery_Cell, symbol Device:Battery_Cell
- added J101: SD Card, Connector_PinSocket_2.54mm:PinSocket_1x08_P2.54mm_Vertical, symbol Connector:Conn_01x08_Female
- added JP101, JP105: PumpAngGND, Jumper:SolderJumper-2_P1.3mm_Open_Pad1.0x1.5mm, symbol Jumper:SolderJumper_2_Open
- added U101: Teensy3.6_All_Pins, Symbol:Teensy35_36, symbol teensy:Teensy3.6_All_Pins
- renumbered JP1 to JP102, JP50 to JP103, JP51 to JP104, R2 to R101, R1 to R102, U1 to U102
Connections:
- net labels added: irid_CTS, irid_NET_AV, irid_RI, irid_RTS, irid_RXD, irid_SLEEP, irid_TXD
- net labels removed: +BATT, -BATT, engine_measured_BATT+, external_switch_A, external_switch_B, lipo_bat1_sense1, lipo_bat1_sense2, lipo_bat1_sense3, lipo_bat1_sense4, lipo_bat1_sense5, lipo_bat1_therm1, lipo_bat1_therm2, lipo_bat_therm1, lipo_bat_therm2, neo08mu_gps_int, neo08mu_gps_pps, neo08mu_gps_rst, neo08mu_gps_safe, pump_measured_BATT+, raw_BATT+, raw_BATT-, rs232_gnd, rs232_rx, rs232_tx, rv1805_sense_int, rv1806_sense_int, rv_1805_sense_psw, solenoid_measured_BATT+, turbine1_blu, turbine1_grn, turbine1_measured_pwr, turbine1_wht, turbine2_blu, turbine2_grn, turbine2_wht, usb_pwr
- wire segments 328 -> 74
Other:
- moved on the sheet: JP102, JP103, JP104, R101, R102, U102

Commit message: pcb parts done, footprints updated, ready for routing
pre-routing step..
- finalized footprints
- verified layout, size, mounting holes (1.75" apart)
Parts:
- added H1, H2, H3, H4, H5, H6, H7, H8: MountingHole, MountingHole:MountingHole_5.3mm_M5_Pad, symbol Mechanical:MountingHole
- added TP101: i2c_sda_1, TestPoint:TestPoint_Loop_D2.60mm_Drill1.6mm_Beaded, symbol engine-board-eagle-import:TEST-POINTTP_15TH_THRU
- added TP102: i2c_scl_1, TestPoint:TestPoint_Loop_D2.60mm_Drill1.6mm_Beaded, symbol engine-board-eagle-import:TEST-POINTTP_15TH_THRU
- BT101: footprint (none) -> Battery:BatteryHolder_Keystone_1060_1x2032
Connections:
- wire segments 74 -> 79
Changed lines of the file:
@@
 F 0 "BT101" H 868 5646 50  0000 L CNN
 F 1 "Battery_Cell" H 868 5555 50  0000 L CNN
-F 2 "" V 750 5610 50  0001 C CNN
+F 2 "Battery:BatteryHolder_Keystone_1060_1x2032" V 750 5610 50  0001 C CNN
 F 3 "~" V 750 5610 50  0001 C CNN
 	1    750  5550
@@
 Text Label 1600 3350 2    50   ~ 0
 turbine_2_pwm
+$Comp
+L engine-board-eagle-import:TEST-POINTTP_15TH_THRU TP101
+U 1 1 61D0D736
+P 4800 7800
+F 0 "TP101" H 4844 8040 70  0000 C CNN
+F 1 "i2c_sda_1" H 4844 7919 70  0000 C CNN
+F 2 "TestPoint:TestPoint_Loop_D2.60mm_Drill1.6mm_Beaded" H 4800 7800 50  0001 C CNN
+F 3 "https://www.keyelco.com/userAssets/file/M65p64.pdf" H 4800 7800 50  0001 C CNN
+F 4 "0.23" H 4800 7800 50  0001 C CNN "Price"
+F 5 "680" H 4800 7800 50  0001 C CNN "MFN"
+F 6 "https://www.digikey.com/en/products/detail/keystone-electronics/680/316581" H 4800 7800 50  0001 C CNN "Link"
+	1    4800 7800
+	1    0    0    -1
+$EndComp
+Wire Wire Line
+	3900 7350 3900 7800
+Wire Wire Line
+	3900 7800 4800 7800
+$Comp
+L engine-board-eagle-import:TEST-POINTTP_15TH_THRU TP102
+U 1 1 61D129F9
+P 5400 7550
+F 0 "TP102" H 5444 7790 70  0000 C CNN
+F 1 "i2c_scl_1" H 5444 7669 70  0000 C CNN
+F 2 "TestPoint:TestPoint_Loop_D2.60mm_Drill1.6mm_Beaded" H 5400 7550 50  0001 C CNN
+F 3 "https://www.keyelco.com/userAssets/file/M65p64.pdf" H 5400 7550 50  0001 C CNN
+F 4 "0.23" H 5400 7550 50  0001 C CNN "Price"
+F 5 "680" H 5400 7550 50  0001 C CNN "MFN"
+F 6 "https://www.digikey.com/en/products/detail/keystone-electronics/680/316581" H 5400 7550 50  0001 C CNN "Link"
+	1    5400 7550
+	1    0    0    -1
+$EndComp
+Wire Wire Line
+	5400 7550 5050 7550
+Wire Wire Line
+	5050 7550 5050 7250
+Wire Wire Line
+	5050 7250 3900 7250
+$Comp
+L Mechanical:MountingHole H1
+U 1 1 61DA7F8F
+P 9650 2450
+F 0 "H1" H 9750 2496 50  0000 L CNN
+F 1 "MountingHole" H 9750 2405 50  0000 L CNN
+F 2 "MountingHole:MountingHole_5.3mm_M5_Pad" H 9650 2450 50  0001 C CNN
+F 3 "~" H 9650 2450 50  0001 C CNN
+	1    9650 2450
+	1    0    0    -1
+$EndComp
+$Comp
+L Mechanical:MountingHole H2
+U 1 1 61DAC0EA
+P 9650 2650
+F 0 "H2" H 9750 2696 50  0000 L CNN
+F 1 "MountingHole" H 9750 2605 50  0000 L CNN
+F 2 "MountingHole:MountingHole_5.3mm_M5_Pad" H 9650 2650 50  0001 C CNN
+F 3 "~" H 9650 2650 50  0001 C CNN
+	1    9650 2650
+	1    0    0    -1
+$EndComp
+$Comp
+L Mechanical:MountingHole H3
+U 1 1 61DAEE2D
+P 9650 2850
+F 0 "H3" H 9750 2896 50  0000 L CNN
+F 1 "MountingHole" H 9750 2805 50  0000 L CNN
+F 2 "MountingHole:MountingHole_5.3mm_M5_Pad" H 9650 2850 50  0001 C CNN
+F 3 "~" H 9650 2850 50  0001 C CNN
+	1    9650 2850
+	1    0    0    -1
+$EndComp
+$Comp
+L Mechanical:MountingHole H4
+U 1 1 61DB1B7F
+P 9650 3050
+F 0 "H4" H 9750 3096 50  0000 L CNN
+F 1 "MountingHole" H 9750 3005 50  0000 L CNN
+F 2 "MountingHole:MountingHole_5.3mm_M5_Pad" H 9650 3050 50  0001 C CNN
+F 3 "~" H 9650 3050 50  0001 C CNN
+	1    9650 3050
+	1    0    0    -1
+$EndComp
+$Comp
+L Mechanical:MountingHole H5
+U 1 1 61DB4859
+P 9650 3250
+F 0 "H5" H 9750 3296 50  0000 L CNN
+F 1 "MountingHole" H 9750 3205 50  0000 L CNN
+F 2 "MountingHole:MountingHole_5.3mm_M5_Pad" H 9650 3250 50  0001 C CNN
+F 3 "~" H 9650 3250 50  0001 C CNN
+	1    9650 3250
+	1    0    0    -1
+$EndComp
+$Comp
+L Mechanical:MountingHole H6
+U 1 1 61DB7527
+P 9650 3450
+F 0 "H6" H 9750 3496 50  0000 L CNN
+F 1 "MountingHole" H 9750 3405 50  0000 L CNN
+F 2 "MountingHole:MountingHole_5.3mm_M5_Pad" H 9650 3450 50  0001 C CNN
+F 3 "~" H 9650 3450 50  0001 C CNN
+	1    9650 3450
+	1    0    0    -1
+$EndComp
+$Comp
+L Mechanical:MountingHole H7
+U 1 1 61DBE384
+P 9650 3650
+F 0 "H7" H 9750 3696 50  0000 L CNN
+F 1 "MountingHole" H 9750 3605 50  0000 L CNN
+F 2 "MountingHole:MountingHole_5.3mm_M5_Pad" H 9650 3650 50  0001 C CNN
+F 3 "~" H 9650 3650 50  0001 C CNN
+	1    9650 3650
+	1    0    0    -1
+$EndComp
+$Comp
+L Mechanical:MountingHole H8
+U 1 1 61DC1124
+P 9650 3850
+F 0 "H8" H 9750 3896 50  0000 L CNN
+F 1 "MountingHole" H 9750 3805 50  0000 L CNN
+F 2 "MountingHole:MountingHole_5.3mm_M5_Pad" H 9650 3850 50  0001 C CNN
+F 3 "~" H 9650 3850 50  0001 C CNN
+	1    9650 3850
+	1    0    0    -1
+$EndComp
 $EndSCHEMATC

Commit message: shortend pcb, ready to route
ready to route, shortend pcb, layout complete
Parts:
- removed H5, H6: MountingHole, MountingHole:MountingHole_5.3mm_M5_Pad, symbol Mechanical:MountingHole
- removed TP101: i2c_sda_1, TestPoint:TestPoint_Loop_D2.60mm_Drill1.6mm_Beaded, symbol engine-board-eagle-import:TEST-POINTTP_15TH_THRU
- removed TP102: i2c_scl_1, TestPoint:TestPoint_Loop_D2.60mm_Drill1.6mm_Beaded, symbol engine-board-eagle-import:TEST-POINTTP_15TH_THRU
Connections:
- net labels removed: 3v3_feather
- wire segments 79 -> 85
Other:
- moved on the sheet: R101, R102
Changed lines of the file:
@@
 L Device:R_Small R102
 U 1 1 60DA427C
-P 6000 6350
-F 0 "R102" V 6196 6350 50  0000 C CNN
-F 1 "33ohm" V 6105 6350 50  0000 C CNN
-F 2 "Resistor_THT:R_Axial_DIN0204_L3.6mm_D1.6mm_P5.08mm_Vertical" H 6000 6350 50  0001 C CNN
-F 3 "~" H 6000 6350 50  0001 C CNN
-	1    6000 6350
+P 6000 6300
+F 0 "R102" V 6196 6300 50  0000 C CNN
+F 1 "33ohm" V 6105 6300 50  0000 C CNN
+F 2 "Resistor_THT:R_Axial_DIN0204_L3.6mm_D1.6mm_P5.08mm_Vertical" H 6000 6300 50  0001 C CNN
+F 3 "~" H 6000 6300 50  0001 C CNN
+	1    6000 6300
 	0    -1   -1   0
 $EndComp
@@
 L Device:R_Small R101
 U 1 1 60DAF797
-P 6000 6050
-F 0 "R101" V 6196 6050 50  0000 C CNN
-F 1 "33ohm" V 6105 6050 50  0000 C CNN
-F 2 "Resistor_THT:R_Axial_DIN0204_L3.6mm_D1.6mm_P5.08mm_Vertical" H 6000 6050 50  0001 C CNN
-F 3 "~" H 6000 6050 50  0001 C CNN
-	1    6000 6050
+P 6000 6000
+F 0 "R101" V 6196 6000 50  0000 C CNN
+F 1 "33ohm" V 6105 6000 50  0000 C CNN
+F 2 "Resistor_THT:R_Axial_DIN0204_L3.6mm_D1.6mm_P5.08mm_Vertical" H 6000 6000 50  0001 C CNN
+F 3 "~" H 6000 6000 50  0001 C CNN
+	1    6000 6000
 	0    -1   -1   0
 $EndComp
@@
 Wire Wire Line
 	8900 5450 9100 5450
-Text Label 8900 4650 0    50   ~ 0
-3v3_feather
 Text Label 9100 5950 0    50   ~ 0
 imu_cs
@@
 turbine_2_pwm
 $Comp
-L engine-board-eagle-import:TEST-POINTTP_15TH_THRU TP101
-U 1 1 61D0D736
-P 4800 7800
-F 0 "TP101" H 4844 8040 70  0000 C CNN
-F 1 "i2c_sda_1" H 4844 7919 70  0000 C CNN
-F 2 "TestPoint:TestPoint_Loop_D2.60mm_Drill1.6mm_Beaded" H 4800 7800 50  0001 C CNN
-F 3 "https://www.keyelco.com/userAssets/file/M65p64.pdf" H 4800 7800 50  0001 C CNN
-F 4 "0.23" H 4800 7800 50  0001 C CNN "Price"
-F 5 "680" H 4800 7800 50  0001 C CNN "MFN"
-F 6 "https://www.digikey.com/en/products/detail/keystone-electronics/680/316581" H 4800 7800 50  0001 C CNN "Link"
-	1    4800 7800
-	1    0    0    -1
-$EndComp
-Wire Wire Line
-	3900 7350 3900 7800
-Wire Wire Line
-	3900 7800 4800 7800
-$Comp
-L engine-board-eagle-import:TEST-POINTTP_15TH_THRU TP102
-U 1 1 61D129F9
-P 5400 7550
-F 0 "TP102" H 5444 7790 70  0000 C CNN
-F 1 "i2c_scl_1" H 5444 7669 70  0000 C CNN
-F 2 "TestPoint:TestPoint_Loop_D2.60mm_Drill1.6mm_Beaded" H 5400 7550 50  0001 C CNN
-F 3 "https://www.keyelco.com/userAssets/file/M65p64.pdf" H 5400 7550 50  0001 C CNN
-F 4 "0.23" H 5400 7550 50  0001 C CNN "Price"
-F 5 "680" H 5400 7550 50  0001 C CNN "MFN"
-F 6 "https://www.digikey.com/en/products/detail/keystone-electronics/680/316581" H 5400 7550 50  0001 C CNN "Link"
-	1    5400 7550
-	1    0    0    -1
-$EndComp
-Wire Wire Line
-	5400 7550 5050 7550
-Wire Wire Line
-	5050 7550 5050 7250
-Wire Wire Line
-	5050 7250 3900 7250
-$Comp
 L Mechanical:MountingHole H1
 U 1 1 61DA7F8F
@@
 $EndComp
 $Comp
-L Mechanical:MountingHole H5
-U 1 1 61DB4859
-P 9650 3250
-F 0 "H5" H 9750 3296 50  0000 L CNN
-F 1 "MountingHole" H 9750 3205 50  0000 L CNN
-F 2 "MountingHole:MountingHole_5.3mm_M5_Pad" H 9650 3250 50  0001 C CNN
-F 3 "~" H 9650 3250 50  0001 C CNN
-	1    9650 3250
-	1    0    0    -1
-$EndComp
-$Comp
-L Mechanical:MountingHole H6
-U 1 1 61DB7527
-P 9650 3450
-F 0 "H6" H 9750 3496 50  0000 L CNN
-F 1 "MountingHole" H 9750 3405 50  0000 L CNN
-F 2 "MountingHole:MountingHole_5.3mm_M5_Pad" H 9650 3450 50  0001 C CNN
-F 3 "~" H 9650 3450 50  0001 C CNN
-	1    9650 3450
-	1    0    0    -1
-$EndComp
-$Comp
 L Mechanical:MountingHole H7
 U 1 1 61DBE384
@@
 	1    0    0    -1
 $EndComp
+Wire Wire Line
+	1600 7350 1600 7550
+Wire Wire Line
+	1600 7250 950  7250
+Wire Wire Line
+	950  7250 950  7600
+Wire Wire Line
+	1600 7150 900  7150
+Wire Wire Line
+	900  7150 900  7650
+Wire Wire Line
+	1600 7050 550  7050
+Wire Wire Line
+	550  7050 550  7700
+Wire Wire Line
+	5900 6050 5900 6000
+Wire Wire Line
+	6100 6050 6100 6000
+Wire Wire Line
+	6100 6350 6100 6300
+Wire Wire Line
+	5900 6350 5900 6300
+Text Label 4600 700  2    50   ~ 0
+usb_data_D0
+Text Label 4600 800  2    50   ~ 0
+usb_data_D1
 $EndSCHEMATC
