File: engine-board/engine-board-sensors.sch (KiCad schematic (older format))
At the start: 14 parts, among them J201 Reservoir Pressure Sensor, J202 Bladder Pressure Sensor, J203 HMC6343 COMPASS, J204 QWIIC 1, J205 QWIIC 2, J206 Leak Sensor, J207 BME260 Sensor, J208 RV1805 Clock, J209 External Pressure Sensor, U201 QuickFit_02x03_Header-Connect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, U202 BN0055 IMU

Commit message: board smaller
PCB V0.1 Errata:

- [QUESTION: - it looks like 12 on website] polulu 2814 has 16 pin footprint instead of 12...  AAACK!!!
- 5v and 3.3v traces could be wider
- [FIXED] fail: going into the power schematic scl + sda are swapped...
- [FIXED - moved to miniofit] pump controller silkscreen is wrong
- [FIXED] NOTE: just switch ALL to the minifit??
- [FIXED - will be on top, but not needed now] ADD: Ethernet connection from the teensy to the host computer board.
- [FIXED - going to use Qwiic) 9 Axis Mopak: wrong footprint - holes too small, spacing seems good, create outline as it bumps into feather header
- [FIXED] RV1805:  power + GND swapped... and I can’t seem to find them.
- [FIXED] 2 pressure sensors, the same i2c address... rerouted to 2nd i2c port on teensy
- [NOT NEEDED - adding display] Add RGB LED... it will be helpful for debugging.
- [FIXED - kindof - moved to micro-fit, might need to wire this directly to bulkhead] Turbine ferrules for power are 12 gauge - need bigger screw terminals if that is the connection method
- [FIXED] Feather footprint - lookup exactly what feather boards need for support..
- [FIXED] pump_motor_pwm is not connected to the TEENSY!!  blerg.  (jumper to pin 13 of feather for now)
- [FIXED - added FET] Maxon 70/30 POWER?  Think about power FET or ‘sleep’ to turn it off.
- [FIXED - added to bulkhead connector] Teensy 4.1 Program + ON/OFF pins - research how to extend these
- [TODO] remove VL6180 range sensor
- [LATER - will add to cost.. possibly remove?] put battery on back side
- add silkscreen for polulu
- [FIXED] Reorganize connectors:
    - Pump motor connectors go on end - attached in closing
    - bulkhead connectors go on side as they will always be attached
Parts:
- J201: Link2 (none) -> https://www.alliedelec.com/product/te-connectivity/m30j1-00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; MATE_Link https://www.digikey.com/en/products/detail/molex/0430250400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 -> https://www.digikey.com/en/products/detail/molex/0430250408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; MATE_MPN 430250400 -> 0430250408; MPN2 (none) -> M30J1-000105-300PG; Price2 0 -> 76.57
- J202: Link2 (none) -> https://www.alliedelec.com/product/te-connectivity/m30j1-00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; MATE_Link https://www.digikey.com/en/products/detail/molex/0430250400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 -> https://www.digikey.com/en/products/detail/molex/0430250408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; MATE_MPN 430250400 -> 0430250408; MPN2 (none) -> M30J1-000105-300PG; Price2 (none) -> 76.57
- J203: Link https://www.digikey.com/en/products/detail/samtec-inc/SSQ-106-01-G-S/1110613 -> https://www.digikey.com/en/products/detail/samtec-inc/SSQ-104-01-G-S/1110615; MPN SSQ-106-01-G-S -> SSQ-104-01-G-S
- J206: footprint TerminalBlock_CUI:CUI_TBP01R1W-508-04BE -> Connector_Molex:Molex_Micro-Fit_3.0_43045-0421_2x02-1MP_P3.00mm_Horizontal; Link2 (none) -> https://bluerobotics.com/store/sensors-sonars-cameras/leak-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; MPN2 (none) -> SOS-SET-R1-RP; Manufacturer (none) -> Blue Robotics; Price2 (none) -> 29
- J207: MATE_Link (none) -> https://www.digikey.com/en/products/detail/molex/0901210124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; MATE_MPN (none) -> 0901210124; MATE_Price (none) -> 0.88; Manufacturer (none) -> Sparkfun
- J208: MATE_Link (none) -> https://www.digikey.com/en/products/detail/molex/0901210127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; MATE_MPN (none) -> 0901210127; MATE_Price (none) -> 1.34; Manufacturer (none) -> Sparkfun
- J209: MATE_Link https://www.digikey.com/en/products/detail/molex/0430250400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 -> https://www.digikey.com/en/products/detail/molex/0430250408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; MATE_MPN 430250400 -> 430250408; MPM2 BAR100-SENSOR-R2-RP -> (none); MPN2 (none) -> BAR100-SENSOR-R2-RP; Manufacturer (none) -> Blue Robotics
- U201: value QuickFit_02x03_Header-Connector -> Bulkhead SW EXT PRESS; MATE_Link (none) -> https://www.digikey.com/en/products/detail/molex/0430250600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; MATE_MPN (none) -> 0430250600; MPM 430450621 -> (none); MPN (none) -> 430450621; Mate_Price (none) -> 0.52
- U202: Link https://www.adafruit.com/product/2472 -> https://www.digikey.com/en/products/detail/samtec-inc/SSQ-1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; Link2 (none) -> https://www.adafruit.com/product/2472; MATE_Link (none) -> https://www.digikey.com/en/products/detail/samtec-inc/SSQ-1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; MATE_MPN (none) -> SSQ-104-01-G-S; MATE_Price (none) -> 0.90; MPM ADA 2472 -> (none); MPN (none) -> SSQ-106-01-G-S; MPN2 (none) -> ADA 2472; Price 34.95 -> 1.35; Price2 (none) -> 34.95
Changed lines of the file:
@@
 F 0 "J206" H 8450 1267 50  0000 C CNN
 F 1 "Leak Sensor" H 8450 1176 50  0000 C CNN
-F 2 "TerminalBlock_CUI:CUI_TBP01R1W-508-04BE" H 8400 1050 50  0001 C CNN
+F 2 "Connector_Molex:Molex_Micro-Fit_3.0_43045-0421_2x02-1MP_P3.00mm_Horizontal" H 8400 1050 50  0001 C CNN
 F 3 "~" H 8400 1050 50  0001 C CNN
 F 4 "https://www.digikey.com/en/products/detail/cui-devices/TBP01R1W-508-04BE/10238427?WT.z_cid=ref_neda_dkc_buynow_cuidevices&utm_source=ecia&utm_medium=aggregator&utm_campaign=cuidevices" H 8400 1050 50  0001 C CNN "Link"
@@
 F 6 "TBP01R1W-508-04BE" H 8400 1050 50  0001 C CNN "MPN"
 F 7 "1.28" H 8400 1050 50  0001 C CNN "Price"
+F 8 "https://bluerobotics.com/store/sensors-sonars-cameras/leak-sensor/sos-leak-sensor/" H 8400 1050 50  0001 C CNN "Link2"
+F 9 "SOS-SET-R1-RP" H 8400 1050 50  0001 C CNN "MPN2"
+F 10 "Blue Robotics" H 8400 1050 50  0001 C CNN "Manufacturer"
+F 11 "29" H 8400 1050 50  0001 C CNN "Price2"
 	1    8400 1050
 	1    0    0    -1
@@
 F 9 "https://www.sparkfun.com/products/14558" H 9250 3200 50  0001 C CNN "Link2"
 F 10 "16.95" H 9250 3200 50  0001 C CNN "Price2"
+F 11 "Sparkfun" H 9250 3200 50  0001 C CNN "Manufacturer"
+F 12 "https://www.digikey.com/en/products/detail/molex/0901210127/760816" H 9250 3200 50  0001 C CNN "MATE_Link"
+F 13 "0901210127" H 9250 3200 50  0001 C CNN "MATE_MPN"
+F 14 "1.34" H 9250 3200 50  0001 C CNN "MATE_Price"
 	1    9250 3200
 	1    0    0    -1
@@
 F 6 "0430450422" H 2050 1450 50  0001 C CNN "MPN"
 F 7 "2.38" H 2050 1450 50  0001 C CNN "Price"
-F 8 "430250400" H 2050 1450 50  0001 C CNN "MATE_MPN"
+F 8 "0430250408" H 2050 1450 50  0001 C CNN "MATE_MPN"
 F 9 "0.48" H 2050 1450 50  0001 C CNN "MATE_Price"
-F 10 "https://www.digikey.com/en/products/detail/molex/0430250400/252497" H 2050 1450 50  0001 C CNN "MATE_Link"
-F 11 "0" H 2050 1450 50  0001 C CNN "Price2"
+F 10 "https://www.digikey.com/en/products/detail/molex/0430250408/4481508?s=N4IgTCBcDaICwGYAMYCsS5IBwgLoF8g" H 2050 1450 50  0001 C CNN "MATE_Link"
+F 11 "76.57" H 2050 1450 50  0001 C CNN "Price2"
+F 12 "https://www.alliedelec.com/product/te-connectivity/m30j1-000105-300pg/71023700/" H 2050 1450 50  0001 C CNN "Link2"
+F 13 "M30J1-000105-300PG" H 2050 1450 50  0001 C CNN "MPN2"
 	1    2050 1450
 	1    0    0    -1
@@
 F 6 "0430450422" H 2050 1900 50  0001 C CNN "MPN"
 F 7 "2.38" H 2050 1900 50  0001 C CNN "Price"
-F 8 "430250400" H 2050 1900 50  0001 C CNN "MATE_MPN"
+F 8 "0430250408" H 2050 1900 50  0001 C CNN "MATE_MPN"
 F 9 "0.48" H 2050 1900 50  0001 C CNN "MATE_Price"
-F 10 "https://www.digikey.com/en/products/detail/molex/0430250400/252497" H 2050 1900 50  0001 C CNN "MATE_Link"
+F 10 "https://www.digikey.com/en/products/detail/molex/0430250408/4481508" H 2050 1900 50  0001 C CNN "MATE_Link"
+F 11 "https://www.alliedelec.com/product/te-connectivity/m30j1-000105-300pg/71023700/" H 2050 1900 50  0001 C CNN "Link2"
+F 12 "M30J1-000105-300PG" H 2050 1900 50  0001 C CNN "MPN2"
+F 13 "76.57" H 2050 1900 50  0001 C CNN "Price2"
 	1    2050 1900
 	1    0    0    -1
@@
 F 2 "Connector_PinSocket_2.54mm:PinSocket_1x04_P2.54mm_Vertical" H 5850 1200 50  0001 C CNN
 F 3 "~" H 5850 1200 50  0001 C CNN
-F 4 "https://www.digikey.com/en/products/detail/samtec-inc/SSQ-106-01-G-S/1110613" H 5850 1200 50  0001 C CNN "Link"
+F 4 "https://www.digikey.com/en/products/detail/samtec-inc/SSQ-104-01-G-S/1110615" H 5850 1200 50  0001 C CNN "Link"
 F 5 "Samtec Inc." H 5850 1200 50  0001 C CNN "MANUFACTURER"
-F 6 "SSQ-106-01-G-S" H 5850 1200 50  0001 C CNN "MPN"
+F 6 "SSQ-104-01-G-S" H 5850 1200 50  0001 C CNN "MPN"
 F 7 "1.35" H 5850 1200 50  0001 C CNN "Price"
 F 8 "ADDR=0x32" H 6100 1250 50  0000 C CNN "I2C_ADDR"
@@
 F 2 "Sensor_Motion:ADA_BN0055" H 6450 4150 50  0001 C CNN
 F 3 "https://www.adafruit.com/product/2472" H 6450 4150 50  0001 C CNN
-F 4 "ADA 2472" H 6450 4150 50  0001 C CNN "MPM"
-F 5 "https://www.adafruit.com/product/2472" H 6450 4150 50  0001 C CNN "Link"
-F 6 "34.95" H 6450 4150 50  0001 C CNN "Price"
+F 4 "" H 6450 4150 50  0001 C CNN "MPM"
+F 5 "https://www.digikey.com/en/products/detail/samtec-inc/SSQ-106-01-G-S/1110613" H 6450 4150 50  0001 C CNN "Link"
+F 6 "1.35" H 6450 4150 50  0001 C CNN "Price"
 F 7 "ADDR=0x28" H 6475 4183 50  0000 C CNN "I2C_ADDR"
+F 8 "SSQ-106-01-G-S" H 6450 4150 50  0001 C CNN "MPN"
+F 9 "https://www.adafruit.com/product/2472" H 6450 4150 50  0001 C CNN "Link2"
+F 10 "ADA 2472" H 6450 4150 50  0001 C CNN "MPN2"
+F 11 "34.95" H 6450 4150 50  0001 C CNN "Price2"
+F 12 "https://www.digikey.com/en/products/detail/samtec-inc/SSQ-104-01-G-S/1110615" H 6450 4150 50  0001 C CNN "MATE_Link"
+F 13 "SSQ-104-01-G-S" H 6450 4150 50  0001 C CNN "MATE_MPN"
+F 14 "0.90" H 6450 4150 50  0001 C CNN "MATE_Price"
 	1    6450 4150
 	1    0    0    -1
@@
 F 9 "https://www.sparkfun.com/products/13676" H 9250 3950 50  0001 C CNN "Link2"
 F 10 "19.95" H 9250 3950 50  0001 C CNN "Price2"
+F 11 "Sparkfun" H 9250 3950 50  0001 C CNN "Manufacturer"
+F 12 "https://www.digikey.com/en/products/detail/molex/0901210124/760813?s=N4IgTCBcDaIJwAYCMYnLAFhAXQL5A" H 9250 3950 50  0001 C CNN "MATE_Link"
+F 13 "0901210124" H 9250 3950 50  0001 C CNN "MATE_MPN"
+F 14 "0.88" H 9250 3950 50  0001 C CNN "MATE_Price"
 	1    9250 3950
 	1    0    0    -1
@@
 AR Path="/618F9F5D/62037C79" Ref="U201"  Part="1"
 F 0 "U201" H 2100 2375 50  0000 C CNN
-F 1 "QuickFit_02x03_Header-Connector" H 2100 2284 50  0000 C CNN
+F 1 "Bulkhead SW EXT PRESS" H 2100 2284 50  0000 C CNN
 F 2 "Connector_Molex:Molex_Micro-Fit_3.0_43045-0621_2x03-1MP_P3.00mm_Horizontal" H 2050 2600 50  0001 C CNN
 F 3 "" H 2050 2600 50  0001 C CNN
 F 4 "https://www.digikey.com/short/4c5hw39j" H 2100 2450 50  0001 C CNN "Link"
-F 5 "430450621" H 2100 2450 50  0001 C CNN "MPM"
+F 5 "0430250600" H 2100 2450 50  0001 C CNN "MATE_MPN"
 F 6 "2.19" H 2100 2450 50  0001 C CNN "Price"
+F 7 "430450621" H 2100 2450 50  0001 C CNN "MPN"
+F 8 "https://www.digikey.com/en/products/detail/molex/0430250600/252498" H 2100 2450 50  0001 C CNN "MATE_Link"
+F 9 "0.52" H 2100 2450 50  0001 C CNN "Mate_Price"
 	1    2100 2450
 	1    0    0    -1
@@
 F 6 "0430450421" H 2150 3500 50  0001 C CNN "MPN"
 F 7 "2.04" H 2150 3500 50  0001 C CNN "Price"
-F 8 "430250400" H 2150 3500 50  0001 C CNN "MATE_MPN"
+F 8 "430250408" H 2150 3500 50  0001 C CNN "MATE_MPN"
 F 9 "0.48" H 2150 3500 50  0001 C CNN "MATE_Price"
-F 10 "https://www.digikey.com/en/products/detail/molex/0430250400/252497" H 2150 3500 50  0001 C CNN "MATE_Link"
+F 10 "https://www.digikey.com/en/products/detail/molex/0430250408/4481508" H 2150 3500 50  0001 C CNN "MATE_Link"
 F 11 "259" H 2150 3500 50  0001 C CNN "Price2"
 F 12 "https://bluerobotics.com/store/sensors-sonars-cameras/sensors/bar100-sensor-r2-rp/" H 2150 3500 50  0001 C CNN "Link2"
-F 13 "BAR100-SENSOR-R2-RP" H 2150 3500 50  0001 C CNN "MPM2"
+F 13 "BAR100-SENSOR-R2-RP" H 2150 3500 50  0001 C CNN "MPN2"
+F 14 "Blue Robotics" H 2150 3500 50  0001 C CNN "Manufacturer"
 	1    2150 3500
 	1    0    0    -1
